Commit message: Add ROS 1 control plugins for Gazebo Classic
Signed-off-by: Andrej Orsula <orsula.andrej@gmail.com>

File: lunalab_summit_xl_gen_description/urdf/lunalab_summit_xl_gen.urdf.xacro (robot description, xacro)
@@ -28,4 +28,10 @@
   <!-- (unimplemented!) Flag to select the high or low quality model -->
   <xacro:arg name="high_quality_mesh" default="ignored"/>
+  <!-- Flag to enable setup of Gazebo ros_planar_move plugin (mobile) -->
+  <xacro:arg name="gazebo_ros_planar_move_plugin" default="false"/>
+  <!-- Flag to enable setup of Gazebo ros_control plugin (manipulation) -->
+  <xacro:arg name="gazebo_ros_control_plugin" default="false"/>
+  <!-- Flag to enable setup of Gazebo ros_ft_sensor plugin (force torque sensor on manipulator joints) -->
+  <xacro:arg name="gazebo_ros_ft_sensor" default="false"/>
   <!--            -->
   <!-- Properties -->
@@ -46,4 +52,5 @@
     add_base_footprint="true"
     high_quality_mesh="$(arg high_quality_mesh)"
+    gazebo_ros_planar_move_plugin="$(arg gazebo_ros_planar_move_plugin)"
   />
   <!-- Kinova Gen2 (Jaco2, spherical wrist, 7DOF, 3-finger gripper) -->
@@ -57,4 +64,6 @@
     safety_k_position="$(arg safety_k_position)"
     high_quality_mesh="$(arg high_quality_mesh)"
+    gazebo_ros_control_plugin="$(arg gazebo_ros_control_plugin)"
+    gazebo_ros_ft_sensor="$(arg gazebo_ros_ft_sensor)"
   />
   <!-- Sensors -->

File: lunalab_summit_xl_gen_description/urdf/lunalab_summit_xl_sensors.xacro (robot description, xacro)
@@ -2,3 +2,40 @@
 <!-- Macro that includes all required sensors -->
 <robot xmlns:xacro="http://wiki.ros.org/xacro">
+  <!-- TODO Use local definition of sensors -->
+  <!-- TODO Add support for all sensors on LunaLab variant with arguments that enable/disable them -->
+  <!--                   -->
+  <!-- Imported elements -->
+  <!--                   -->
+  <!-- Sensors -->
+  <xacro:include filename="$(find robotnik_sensors)/urdf/all_sensors.urdf.xacro"/>
+  <!--       -->
+  <!-- Macro -->
+  <!--       -->
+  <!-- prefix - Prefix for all entities -->
+  <xacro:macro name="lunalab_summit_xl_sensors" params="prefix">
+    <!-- IMU -->
+    <xacro:sensor_imu prefix="$(arg prefix)imu" parent="$(arg prefix)base_link">
+      <origin xyz="-0.18 0.0 0.170" rpy="0 0 0"/>
+    </xacro:sensor_imu>
+    <!-- 2d laser -->
+    <xacro:sensor_hokuyo_ust10lx prefix="$(arg prefix)front_laser" parent="$(arg prefix)base_link" prefix_topic="front_laser" gpu="$(arg gpu)">
+      <origin xyz="0.0 0.0 0.33" rpy="0 0 0"/>
+    </xacro:sensor_hokuyo_ust10lx>
+    <!-- 3d laser -->
+    <xacro:sensor_rslidar_mems prefix="$(arg prefix)top_3d_laser" parent="$(arg prefix)base_link">
+      <origin xyz="0.3134 0 0.2424" rpy="0 0 0"/>
+    </xacro:sensor_rslidar_mems>
+    <!-- ptz camera -->
+    <xacro:sensor_axis prefix="$(arg prefix)front_ptz_camera" parent="$(arg prefix)base_link">
+      <origin xyz="0.19 0 0.26" rpy="0 ${15*pi/180} 0"/>
+    </xacro:sensor_axis>
+    <!-- RGBD -->
+    <xacro:sensor_orbbec_astra prefix="$(arg prefix)front_rgbd_camera" parent="$(arg prefix)base_link" prefix_topic="front_rgbd_camera">
+      <origin xyz="0.324 0.012 0.172" rpy="0 0 0"/>
+    </xacro:sensor_orbbec_astra>
+    <!-- GPS -->
+    <xacro:sensor_gps prefix="$(arg prefix)gps" parent="$(arg prefix)base_link">
+      <origin xyz="-0.28 0 0.6676" rpy="0 0 0"/>
+    </xacro:sensor_gps>
+  </xacro:macro>
 </robot>

File: lunalab_summit_xl_gen_description/urdf/manipulators/kinova/j2s7s300.xacro (robot description, xacro)
@@ -132,23 +132,29 @@
     safety_k_position:=20.0
     high_quality_mesh:=false
+    gazebo_ros_control_plugin:=false
+    gazebo_ros_ft_sensor:=false
   ">
     <xacro:kinova_armlink link_name="${prefix}link_base" link_mesh="${link_base_mesh}" mu="${link_base_mu}"/>
-    <xacro:kinova_armjoint joint_name="${prefix}joint_base" type="${joint_base_type}" parent="${base_parent}" child="${prefix}link_base" joint_axis_xyz="${joint_base_axis_xyz}" joint_origin_xyz="${joint_base_origin_xyz}" joint_origin_rpy="${joint_base_origin_rpy}" joint_lower_limit="0" joint_upper_limit="0" joint_velocity_limit="0" joint_torque_limit="0" fixed="true" safety_limits="${safety_limits}" safety_position_margin="${safety_position_margin}" safety_k_position="${safety_k_position}"/>
+    <xacro:kinova_armjoint joint_name="${prefix}joint_base" type="${joint_base_type}" parent="${base_parent}" child="${prefix}link_base" joint_axis_xyz="${joint_base_axis_xyz}" joint_origin_xyz="${joint_base_origin_xyz}" joint_origin_rpy="${joint_base_origin_rpy}" joint_lower_limit="0" joint_upper_limit="0" joint_velocity_limit="0" joint_torque_limit="0" fixed="true" safety_limits="${safety_limits}" safety_position_margin="${safety_position_margin}" safety_k_position="${safety_k_position}" gazebo_ros_ft_sensor="${gazebo_ros_ft_sensor}"/>
     <xacro:kinova_armlink link_name="${prefix}link_1" link_mesh="${link_1_mesh}" use_ring_mesh="true" mu="${link_1_mu}"/>
-    <xacro:kinova_armjoint joint_name="${prefix}joint_1" type="${joint_1_type}" parent="${prefix}link_base" child="${prefix}link_1" joint_axis_xyz="${joint_1_axis_xyz}" joint_origin_xyz="${joint_1_origin_xyz}" joint_origin_rpy="${joint_1_origin_rpy}" joint_damping="${joint_1_damping}" joint_friction="${joint_1_friction}" joint_lower_limit="${joint_1_lower_limit}" joint_upper_limit="${joint_1_upper_limit}" joint_velocity_limit="${joint_1_velocity_limit}" joint_torque_limit="${joint_1_torque_limit}" safety_limits="${safety_limits}" safety_position_margin="${safety_position_margin}" safety_k_position="${safety_k_position}"/>
+    <xacro:kinova_armjoint joint_name="${prefix}joint_1" type="${joint_1_type}" parent="${prefix}link_base" child="${prefix}link_1" joint_axis_xyz="${joint_1_axis_xyz}" joint_origin_xyz="${joint_1_origin_xyz}" joint_origin_rpy="${joint_1_origin_rpy}" joint_damping="${joint_1_damping}" joint_friction="${joint_1_friction}" joint_lower_limit="${joint_1_lower_limit}" joint_upper_limit="${joint_1_upper_limit}" joint_velocity_limit="${joint_1_velocity_limit}" joint_torque_limit="${joint_1_torque_limit}" safety_limits="${safety_limits}" safety_position_margin="${safety_position_margin}" safety_k_position="${safety_k_position}" gazebo_ros_ft_sensor="${gazebo_ros_ft_sensor}"/>
     <xacro:kinova_armlink link_name="${prefix}link_2" link_mesh="${link_2_mesh}" use_ring_mesh="true" mu="${link_2_mu}"/>
-    <xacro:kinova_armjoint joint_name="${prefix}joint_2" type="${joint_2_type}" parent="${prefix}link_1" child="${prefix}link_2" joint_axis_xyz="${joint_2_axis_xyz}" joint_origin_xyz="${joint_2_origin_xyz}" joint_origin_rpy="${joint_2_origin_rpy}" joint_damping="${joint_2_damping}" joint_friction="${joint_2_friction}" joint_lower_limit="${joint_2_lower_limit}" joint_upper_limit="${joint_2_upper_limit}" joint_velocity_limit="${joint_2_velocity_limit}" joint_torque_limit="${joint_2_torque_limit}" safety_limits="${safety_limits}" safety_position_margin="${safety_position_margin}" safety_k_position="${safety_k_position}"/>
+    <xacro:kinova_armjoint joint_name="${prefix}joint_2" type="${joint_2_type}" parent="${prefix}link_1" child="${prefix}link_2" joint_axis_xyz="${joint_2_axis_xyz}" joint_origin_xyz="${joint_2_origin_xyz}" joint_origin_rpy="${joint_2_origin_rpy}" joint_damping="${joint_2_damping}" joint_friction="${joint_2_friction}" joint_lower_limit="${joint_2_lower_limit}" joint_upper_limit="${joint_2_upper_limit}" joint_velocity_limit="${joint_2_velocity_limit}" joint_torque_limit="${joint_2_torque_limit}" safety_limits="${safety_limits}" safety_position_margin="${safety_position_margin}" safety_k_position="${safety_k_position}" gazebo_ros_ft_sensor="${gazebo_ros_ft_sensor}"/>
     <xacro:kinova_armlink link_name="${prefix}link_3" link_mesh="${link_3_mesh}" use_ring_mesh="true" mu="${link_3_mu}"/>
-    <xacro:kinova_armjoint joint_name="${prefix}joint_3" type="${joint_3_type}" parent="${prefix}link_2" child="${prefix}link_3" joint_axis_xyz="${joint_3_axis_xyz}" joint_origin_xyz="${joint_3_origin_xyz}" joint_origin_rpy="${joint_3_origin_rpy}" joint_damping="${joint_3_damping}" joint_friction="${joint_3_friction}" joint_lower_limit="${joint_3_lower_limit}" joint_upper_limit="${joint_3_upper_limit}" joint_velocity_limit="${joint_3_velocity_limit}" joint_torque_limit="${joint_3_torque_limit}" safety_limits="${safety_limits}" safety_position_margin="${safety_position_margin}" safety_k_position="${safety_k_position}"/>
+    <xacro:kinova_armjoint joint_name="${prefix}joint_3" type="${joint_3_type}" parent="${prefix}link_2" child="${prefix}link_3" joint_axis_xyz="${joint_3_axis_xyz}" joint_origin_xyz="${joint_3_origin_xyz}" joint_origin_rpy="${joint_3_origin_rpy}" joint_damping="${joint_3_damping}" joint_friction="${joint_3_friction}" joint_lower_limit="${joint_3_lower_limit}" joint_upper_limit="${joint_3_upper_limit}" joint_velocity_limit="${joint_3_velocity_limit}" joint_torque_limit="${joint_3_torque_limit}" safety_limits="${safety_limits}" safety_position_margin="${safety_position_margin}" safety_k_position="${safety_k_position}" gazebo_ros_ft_sensor="${gazebo_ros_ft_sensor}"/>
     <xacro:kinova_armlink link_name="${prefix}link_4" link_mesh="${link_4_mesh}" use_ring_mesh="true" mu="${link_4_mu}"/>
-    <xacro:kinova_armjoint joint_name="${prefix}joint_4" type="${joint_4_type}" parent="${prefix}link_3" child="${prefix}link_4" joint_axis_xyz="${joint_4_axis_xyz}" joint_origin_xyz="${joint_4_origin_xyz}" joint_origin_rpy="${joint_4_origin_rpy}" joint_damping="${joint_4_damping}" joint_friction="${joint_4_friction}" joint_lower_limit="${joint_4_lower_limit}" joint_upper_limit="${joint_4_upper_limit}" joint_velocity_limit="${joint_4_velocity_limit}" joint_torque_limit="${joint_4_torque_limit}" safety_limits="${safety_limits}" safety_position_margin="${safety_position_margin}" safety_k_position="${safety_k_position}"/>
+    <xacro:kinova_armjoint joint_name="${prefix}joint_4" type="${joint_4_type}" parent="${prefix}link_3" child="${prefix}link_4" joint_axis_xyz="${joint_4_axis_xyz}" joint_origin_xyz="${joint_4_origin_xyz}" joint_origin_rpy="${joint_4_origin_rpy}" joint_damping="${joint_4_damping}" joint_friction="${joint_4_friction}" joint_lower_limit="${joint_4_lower_limit}" joint_upper_limit="${joint_4_upper_limit}" joint_velocity_limit="${joint_4_velocity_limit}" joint_torque_limit="${joint_4_torque_limit}" safety_limits="${safety_limits}" safety_position_margin="${safety_position_margin}" safety_k_position="${safety_k_position}" gazebo_ros_ft_sensor="${gazebo_ros_ft_sensor}"/>
     <xacro:kinova_armlink link_name="${prefix}link_5" link_mesh="${link_5_mesh}" use_ring_mesh="true" ring_mesh="ring_small" mu="${link_5_mu}"/>
-    <xacro:kinova_armjoint joint_name="${prefix}joint_5" type="${joint_5_type}" parent="${prefix}link_4" child="${prefix}link_5" joint_axis_xyz="${joint_5_axis_xyz}" joint_origin_xyz="${joint_5_origin_xyz}" joint_origin_rpy="${joint_5_origin_rpy}" joint_damping="${joint_5_damping}" joint_friction="${joint_5_friction}" joint_lower_limit="${joint_5_lower_limit}" joint_upper_limit="${joint_5_upper_limit}" joint_velocity_limit="${joint_5_velocity_limit}" joint_torque_limit="${joint_5_torque_limit}" safety_limits="${safety_limits}" safety_position_margin="${safety_position_margin}" safety_k_position="${safety_k_position}"/>
+    <xacro:kinova_armjoint joint_name="${prefix}joint_5" type="${joint_5_type}" parent="${prefix}link_4" child="${prefix}link_5" joint_axis_xyz="${joint_5_axis_xyz}" joint_origin_xyz="${joint_5_origin_xyz}" joint_origin_rpy="${joint_5_origin_rpy}" joint_damping="${joint_5_damping}" joint_friction="${joint_5_friction}" joint_lower_limit="${joint_5_lower_limit}" joint_upper_limit="${joint_5_upper_limit}" joint_velocity_limit="${joint_5_velocity_limit}" joint_torque_limit="${joint_5_torque_limit}" safety_limits="${safety_limits}" safety_position_margin="${safety_position_margin}" safety_k_position="${safety_k_position}" gazebo_ros_ft_sensor="${gazebo_ros_ft_sensor}"/>
     <xacro:kinova_armlink link_name="${prefix}link_6" link_mesh="${link_6_mesh}" use_ring_mesh="true" ring_mesh="ring_small" mu="${link_6_mu}"/>
-    <xacro:kinova_armjoint joint_name="${prefix}joint_6" type="${joint_6_type}" parent="${prefix}link_5" child="${prefix}link_6" joint_axis_xyz="${joint_6_axis_xyz}" joint_origin_xyz="${joint_6_origin_xyz}" joint_origin_rpy="${joint_6_origin_rpy}" joint_damping="${joint_6_damping}" joint_friction="${joint_6_friction}" joint_lower_limit="${joint_6_lower_limit}" joint_upper_limit="${joint_6_upper_limit}" joint_velocity_limit="${joint_6_velocity_limit}" joint_torque_limit="${joint_6_torque_limit}" safety_limits="${safety_limits}" safety_position_margin="${safety_position_margin}" safety_k_position="${safety_k_position}"/>
+    <xacro:kinova_armjoint joint_name="${prefix}joint_6" type="${joint_6_type}" parent="${prefix}link_5" child="${prefix}link_6" joint_axis_xyz="${joint_6_axis_xyz}" joint_origin_xyz="${joint_6_origin_xyz}" joint_origin_rpy="${joint_6_origin_rpy}" joint_damping="${joint_6_damping}" joint_friction="${joint_6_friction}" joint_lower_limit="${joint_6_lower_limit}" joint_upper_limit="${joint_6_upper_limit}" joint_velocity_limit="${joint_6_velocity_limit}" joint_torque_limit="${joint_6_torque_limit}" safety_limits="${safety_limits}" safety_position_margin="${safety_position_margin}" safety_k_position="${safety_k_position}" gazebo_ros_ft_sensor="${gazebo_ros_ft_sensor}"/>
     <xacro:kinova_armlink link_name="${prefix}link_7" link_mesh="${link_7_mesh}" use_ring_mesh="true" ring_mesh="ring_small" mu="${link_7_mu}"/>
-    <xacro:kinova_armjoint joint_name="${prefix}joint_7" type="${joint_7_type}" parent="${prefix}link_6" child="${prefix}link_7" joint_axis_xyz="${joint_7_axis_xyz}" joint_origin_xyz="${joint_7_origin_xyz}" joint_origin_rpy="${joint_7_origin_rpy}" joint_damping="${joint_7_damping}" joint_friction="${joint_7_friction}" joint_lower_limit="${joint_7_lower_limit}" joint_upper_limit="${joint_7_upper_limit}" joint_velocity_limit="${joint_7_velocity_limit}" joint_torque_limit="${joint_7_torque_limit}" safety_limits="${safety_limits}" safety_position_margin="${safety_position_margin}" safety_k_position="${safety_k_position}"/>
+    <xacro:kinova_armjoint joint_name="${prefix}joint_7" type="${joint_7_type}" parent="${prefix}link_6" child="${prefix}link_7" joint_axis_xyz="${joint_7_axis_xyz}" joint_origin_xyz="${joint_7_origin_xyz}" joint_origin_rpy="${joint_7_origin_rpy}" joint_damping="${joint_7_damping}" joint_friction="${joint_7_friction}" joint_lower_limit="${joint_7_lower_limit}" joint_upper_limit="${joint_7_upper_limit}" joint_velocity_limit="${joint_7_velocity_limit}" joint_torque_limit="${joint_7_torque_limit}" safety_limits="${safety_limits}" safety_position_margin="${safety_position_margin}" safety_k_position="${safety_k_position}" gazebo_ros_ft_sensor="${gazebo_ros_ft_sensor}"/>
     <xacro:kinova_virtual_fixed_link joint_name="${prefix}joint_end_effector" parent="${prefix}link_7" child="${prefix}end_effector" joint_origin_xyz="${joint_end_effector_origin_xyz}" joint_origin_rpy="${joint_end_effector_origin_rpy}"/>
     <xacro:kinova_3fingers link_hand="${prefix}link_7" prefix="${prefix}"/>
+    <!-- Add ros_control Gazebo plugin, if enabled -->
+    <xacro:if value="${gazebo_ros_control_plugin}">
+      <xacro:gazebo_ros_control robot_namespace="${prefix}"/>
+    </xacro:if>
   </xacro:macro>
 </robot>

File: lunalab_summit_xl_gen_description/urdf/manipulators/kinova/kinova_common.xacro (robot description, xacro)
@@ -76,4 +76,5 @@
     safety_position_margin:=${10*pi/180}
     safety_k_position:=20.0
+    gazebo_ros_ft_sensor:=false
   ">
     <xacro:if value="${(type == 'fixed' and not fixed) or (type != 'fixed' and fixed)}">
@@ -123,4 +124,8 @@
         </actuator>
       </transmission>
+      <!-- Add ros_ft_sensor Gazebo plugin (torce-torque sensor), if enabled -->
+      <xacro:if value="${gazebo_ros_ft_sensor}">
+        <xacro:gazebo_ros_ft_sensor joint_name="${joint_name}"/>
+      </xacro:if>
     </xacro:unless>
   </xacro:macro>

File: lunalab_summit_xl_gen_description/urdf/summit_xl/summit_xl.xacro (robot description, xacro)
@@ -21,4 +21,5 @@
   <!-- prefix                        - Prefix for all entities -->
   <!-- add_base_footprint            - Flag that enables base footprint link -->
+  <!-- gazebo_ros_planar_move_plugin - Flag to enable setup of Gazebo ros_planar_move plugin (mobile) -->
   <!-- high_quality_mesh             - Flag to select the high or low quality model -->
   <xacro:macro name="summit_xl" params="
@@ -26,4 +27,5 @@
     add_base_footprint:=true
     high_quality_mesh:=true
+    gazebo_ros_planar_move_plugin:=false
   ">
     <!-- Radius of wheels based on the utilised wheels (only default rubber wheels are currently supported) -->
@@ -44,4 +46,8 @@
       <origin xyz="-${wheel_offset_x} -${wheel_offset_y} ${wheel_offset_z}" rpy="0 0 0"/>
     </xacro:rubber_wheel>
+    <!-- Add ros_planar_move Gazebo plugin, if enabled -->
+    <xacro:if value="${gazebo_ros_planar_move_plugin}">
+      <xacro:gazebo_ros_planar_move prefix="${prefix}" publish_tf="true"/>
+    </xacro:if>
   </xacro:macro>
 </robot>

Commit message: Add ros2_control to description - Add spring stiffness to finger tips
Signed-off-by: Andrej Orsula <orsula.andrej@gmail.com>

File: lunalab_summit_xl_gen_description/urdf/lunalab_summit_xl_gen.urdf.xacro (robot description, xacro)
@@ -28,4 +28,6 @@
   <!-- (unimplemented!) Flag to select the high or low quality model -->
   <xacro:arg name="high_quality_mesh" default="ignored"/>
+  <!-- Flag to enable ros2 controllers for manipulator -->
+  <xacro:arg name="ros2_control" default="true"/>
   <!--            -->
   <!-- Properties -->
@@ -57,4 +59,5 @@
     safety_k_position="$(arg safety_k_position)"
     high_quality_mesh="$(arg high_quality_mesh)"
+    ros2_control="$(arg ros2_control)"
   />
   <!-- Sensors -->

File: lunalab_summit_xl_gen_description/urdf/manipulators/kinova/j2s7s300.xacro (robot description, xacro)
@@ -16,4 +16,5 @@
   <xacro:include filename="$(find lunalab_summit_xl_gen_description)/urdf/manipulators/kinova/kinova_finger_set.xacro"/>
   <xacro:include filename="$(find lunalab_summit_xl_gen_description)/urdf/manipulators/kinova/kinova.gazebo"/>
+  <xacro:include filename="$(find lunalab_summit_xl_gen_description)/urdf/manipulators/kinova/kinova.ros2_control"/>
   <!--            -->
   <!-- Properties -->
@@ -132,4 +133,5 @@
     safety_k_position:=20.0
     high_quality_mesh:=false
+    ros2_control:=true
   ">
     <xacro:kinova_armlink link_name="${prefix}link_base" link_mesh="${link_base_mesh}" mu="${link_base_mu}"/>
@@ -151,4 +153,9 @@
     <xacro:kinova_virtual_fixed_link joint_name="${prefix}joint_end_effector" parent="${prefix}link_7" child="${prefix}end_effector" joint_origin_xyz="${joint_end_effector_origin_xyz}" joint_origin_rpy="${joint_end_effector_origin_rpy}"/>
     <xacro:kinova_3fingers link_hand="${prefix}link_7" prefix="${prefix}"/>
+    <!-- ROS 2 control -->
+    <xacro:if value="${ros2_control}">
+      <xacro:ros2_control_j2s7s300_arm name="KinovaArmFakeSystem" prefix="${prefix}"/>
+      <xacro:ros2_control_3fingers name="KinovaGripperFakeSystem" prefix="${prefix}"/>
+    </xacro:if>
   </xacro:macro>
 </robot>

File: lunalab_summit_xl_gen_description/urdf/manipulators/kinova/kinova_finger_set.xacro (robot description, xacro)
@@ -37,6 +37,8 @@
   <xacro:property name="finger_distal_velocity_limit" value="1.0"/>
   <xacro:property name="finger_distal_torque_limit" value="2.0"/>
-  <xacro:property name="finger_distal_damping" value="0.5"/>
-  <xacro:property name="finger_distal_friction" value="0.05"/>
+  <xacro:property name="finger_distal_damping" value="0.05"/>
+  <xacro:property name="finger_distal_friction" value="0.01"/>
+  <xacro:property name="finger_distal_spring_stiffness" value="0.2"/>
+  <xacro:property name="finger_distal_spring_reference" value="0.0"/>
   <xacro:property name="finger_link_distal_mu" value="1.6"/>
   <!--       -->
@@ -109,4 +111,8 @@
       </actuator>
     </transmission>
+    <gazebo reference="${prefix}joint_finger_tip_${finger_number}">
+      <springStiffness value="${finger_distal_spring_stiffness}"/>
+      <springReference value="${finger_distal_spring_reference}"/>
+    </gazebo>
   </xacro:macro>
 </robot>
