Commit message: Add xacros for Ignition Gazebo plugins - DiffDrive - JointTrajectoryController - JointStatePublisher - PosePublisher
Signed-off-by: Andrej Orsula <orsula.andrej@gmail.com>

File: lunalab_summit_xl_gen_description/urdf/lunalab_summit_xl_gen.urdf.xacro (robot description, xacro)
@@ -13,4 +13,6 @@
   <!-- Miscellaneous -->
   <!-- <xacro:include filename="$(find lunalab_summit_xl_gen_description)/urdf/lunalab_summit_xl_misc.xacro"/> -->
+  <!-- Gazebo plugins -->
+  <xacro:include filename="$(find lunalab_summit_xl_gen_description)/urdf/lunalab_summit_xl_gen.gazebo"/>
   <!--            -->
   <!-- Parameters -->
@@ -30,4 +32,12 @@
   <!-- Flag to enable ros2 controllers for manipulator -->
   <xacro:arg name="ros2_control" default="true"/>
+  <!-- Flag to enable DiffDrive Gazebo plugin for Summit XL -->
+  <xacro:arg name="gazebo_diff_drive" default="true"/>
+  <!-- Flag to enable JointTrajectoryController Gazebo plugin for manipulator -->
+  <xacro:arg name="gazebo_joint_trajectory_controller" default="true"/>
+  <!-- Flag to enable JointStatePublisher Gazebo plugin for all joints -->
+  <xacro:arg name="gazebo_joint_state_publisher" default="true"/>
+  <!-- Flag to enable PosePublisher Gazebo plugin for true pose of robot -->
+  <xacro:arg name="gazebo_pose_publisher" default="true"/>
   <!--            -->
   <!-- Properties -->
@@ -40,4 +50,7 @@
   <xacro:property name="manipulator_offset_p" value="0.0"/>
   <xacro:property name="manipulator_offset_y" value="0.0"/>
+  <!-- Prefixes -->
+  <xacro:property name="prefix_summit_xl" value="$(arg prefix)summit_xl_"/>
+  <xacro:property name="prefix_manipulator" value="$(arg prefix)j2s7s300_"/>
   <!--       -->
   <!-- Robot -->
@@ -45,12 +58,13 @@
   <!-- Summit XL -->
   <xacro:summit_xl
-    prefix="$(arg prefix)summit_xl_"
+    prefix="${prefix_summit_xl}"
     add_base_footprint="true"
     high_quality_mesh="$(arg high_quality_mesh)"
+    gazebo_diff_drive="$(arg gazebo_diff_drive)"
   />
   <!-- Kinova Gen2 (Jaco2, spherical wrist, 7DOF, 3-finger gripper) -->
   <xacro:j2s7s300
-    base_parent="$(arg prefix)summit_xl_base_link"
-    prefix="$(arg prefix)j2s7s300_"
+    base_parent="${prefix_summit_xl}base_link"
+    prefix="${prefix_manipulator}"
     joint_base_origin_xyz="${manipulator_offset_x} ${manipulator_offset_y} ${manipulator_offset_z}"
     joint_base_origin_rpy="${manipulator_offset_r} ${manipulator_offset_p} ${manipulator_offset_y}"
@@ -60,4 +74,5 @@
     high_quality_mesh="$(arg high_quality_mesh)"
     ros2_control="$(arg ros2_control)"
+    gazebo_joint_trajectory_controller="$(arg gazebo_joint_trajectory_controller)"
   />
   <!-- Sensors -->
@@ -65,3 +80,11 @@
   <!-- Miscellaneous -->
   <!-- <xacro:lunalab_summit_xl_misc prefix="$(arg prefix)"/> -->
+  <!-- Gazebo - Joint state publisher -->
+  <xacro:if value="$(arg gazebo_joint_state_publisher)">
+    <xacro:gazebo_joint_state_publisher_summit_xl_gen_j2s7s300 prefix_summit_xl="${prefix_summit_xl}" prefix_manipulator="${prefix_manipulator}"/>
+  </xacro:if>
+  <!-- Gazebo - Pose publisher -->
+  <xacro:if value="$(arg gazebo_pose_publisher)">
+    <xacro:gazebo_pose_publisher/>
+  </xacro:if>
 </robot>

File: lunalab_summit_xl_gen_description/urdf/manipulators/kinova/j2s7s300.xacro (robot description, xacro)
@@ -15,6 +15,6 @@
   <xacro:include filename="$(find lunalab_summit_xl_gen_description)/urdf/manipulators/kinova/kinova_common.xacro"/>
   <xacro:include filename="$(find lunalab_summit_xl_gen_description)/urdf/manipulators/kinova/kinova_finger_set.xacro"/>
+  <xacro:include filename="$(find lunalab_summit_xl_gen_description)/urdf/manipulators/kinova/kinova.ros2_control"/>
   <xacro:include filename="$(find lunalab_summit_xl_gen_description)/urdf/manipulators/kinova/kinova.gazebo"/>
-  <xacro:include filename="$(find lunalab_summit_xl_gen_description)/urdf/manipulators/kinova/kinova.ros2_control"/>
   <!--            -->
   <!-- Properties -->
@@ -134,4 +134,5 @@
     high_quality_mesh:=false
     ros2_control:=true
+    gazebo_joint_trajectory_controller:=true
   ">
     <xacro:kinova_armlink link_name="${prefix}link_base" link_mesh="${link_base_mesh}" mu="${link_base_mu}"/>
@@ -158,4 +159,8 @@
       <xacro:ros2_control_3fingers name="KinovaGripperFakeSystem" prefix="${prefix}"/>
     </xacro:if>
+    <!-- Gazebo - Joint trajectory controller -->
+    <xacro:if value="${gazebo_joint_trajectory_controller}">
+      <xacro:gazebo_joint_trajectory_controller_j2s7s300 prefix="${prefix}"/>
+    </xacro:if>
   </xacro:macro>
 </robot>

File: lunalab_summit_xl_gen_description/urdf/summit_xl/summit_xl.xacro (robot description, xacro)
@@ -9,4 +9,6 @@
   <!-- Import Summit XL wheels (rubber) -->
   <xacro:include filename="$(find lunalab_summit_xl_gen_description)/urdf/summit_xl/rubber_wheel.xacro"/>
+  <!-- Gazebo plugins -->
+  <xacro:include filename="$(find lunalab_summit_xl_gen_description)/urdf/summit_xl/summit_xl.gazebo"/>
   <!--            -->
   <!-- Properties -->
@@ -26,4 +28,5 @@
     add_base_footprint:=true
     high_quality_mesh:=true
+    gazebo_diff_drive:=true
   ">
     <!-- Radius of wheels based on the utilised wheels (only default rubber wheels are currently supported) -->
@@ -44,4 +47,8 @@
       <origin xyz="-${wheel_offset_x} -${wheel_offset_y} ${wheel_offset_z}" rpy="0 0 0"/>
     </xacro:rubber_wheel>
+    <!-- Gazebo - Differential drive -->
+    <xacro:if value="${gazebo_diff_drive}">
+      <xacro:gazebo_diff_drive prefix="${prefix}" wheel_separation="${2*wheel_offset_y}" wheel_radius="${wheel_radius}"/>
+    </xacro:if>
   </xacro:macro>
 </robot>

File: lunalab_summit_xl_gen_description/urdf/summit_xl/summit_xl_base.xacro (robot description, xacro)
@@ -1,8 +1,4 @@
 <?xml version="1.0"?>
 <robot xmlns:xacro="http://wiki.ros.org/xacro">
-  <!--                   -->
-  <!-- Imported elements -->
-  <!--                   -->
-  <xacro:include filename="$(find lunalab_summit_xl_gen_description)/urdf/summit_xl/summit.gazebo"/>
   <!--       -->
   <!-- Macro -->
