Commit message: Add gazebo_preserve_fixed_joint xacro argument
Signed-off-by: Andrej Orsula <orsula.andrej@gmail.com>

File: lunalab_summit_xl_gen_description/urdf/lunalab_summit_xl_gen.urdf.xacro (robot description, xacro)
@@ -32,4 +32,6 @@
   <!-- Flag to enable ros2 controllers for manipulator -->
   <xacro:arg name="ros2_control" default="true"/>
+  <!-- Flag to preserve fixed joints and prevent lumping when generating SDF for Gazebo -->
+  <xacro:arg name="gazebo_preserve_fixed_joint" default="false"/>
   <!-- Flag to enable DiffDrive Gazebo plugin for Summit XL -->
   <xacro:arg name="gazebo_diff_drive" default="true"/>
@@ -61,4 +63,5 @@
     add_base_footprint="true"
     high_quality_mesh="$(arg high_quality_mesh)"
+    gazebo_preserve_fixed_joint="$(arg gazebo_preserve_fixed_joint)"
     gazebo_diff_drive="$(arg gazebo_diff_drive)"
   />
@@ -74,4 +77,5 @@
     high_quality_mesh="$(arg high_quality_mesh)"
     ros2_control="$(arg ros2_control)"
+    gazebo_preserve_fixed_joint="$(arg gazebo_preserve_fixed_joint)"
     gazebo_joint_trajectory_controller="$(arg gazebo_joint_trajectory_controller)"
   />

File: lunalab_summit_xl_gen_description/urdf/manipulators/kinova/j2s7s300.xacro (robot description, xacro)
@@ -134,23 +134,24 @@
     high_quality_mesh:=false
     ros2_control:=true
+    gazebo_preserve_fixed_joint:=false
     gazebo_joint_trajectory_controller:=true
   ">
     <xacro:kinova_armlink link_name="${prefix}link_base" link_mesh="${link_base_mesh}" mu="${link_base_mu}"/>
-    <xacro:kinova_armjoint joint_name="${prefix}joint_base" type="${joint_base_type}" parent="${base_parent}" child="${prefix}link_base" joint_axis_xyz="${joint_base_axis_xyz}" joint_origin_xyz="${joint_base_origin_xyz}" joint_origin_rpy="${joint_base_origin_rpy}" joint_lower_limit="0" joint_upper_limit="0" joint_velocity_limit="0" joint_torque_limit="0" fixed="true" safety_limits="${safety_limits}" safety_position_margin="${safety_position_margin}" safety_k_position="${safety_k_position}"/>
+    <xacro:kinova_armjoint joint_name="${prefix}joint_base" type="${joint_base_type}" parent="${base_parent}" child="${prefix}link_base" joint_axis_xyz="${joint_base_axis_xyz}" joint_origin_xyz="${joint_base_origin_xyz}" joint_origin_rpy="${joint_base_origin_rpy}" joint_lower_limit="0" joint_upper_limit="0" joint_velocity_limit="0" joint_torque_limit="0" fixed="true" safety_limits="${safety_limits}" safety_position_margin="${safety_position_margin}" safety_k_position="${safety_k_position}" gazebo_preserve_fixed_joint="${gazebo_preserve_fixed_joint}"/>
     <xacro:kinova_armlink link_name="${prefix}link_1" link_mesh="${link_1_mesh}" use_ring_mesh="true" mu="${link_1_mu}"/>
-    <xacro:kinova_armjoint joint_name="${prefix}joint_1" type="${joint_1_type}" parent="${prefix}link_base" child="${prefix}link_1" joint_axis_xyz="${joint_1_axis_xyz}" joint_origin_xyz="${joint_1_origin_xyz}" joint_origin_rpy="${joint_1_origin_rpy}" joint_damping="${joint_1_damping}" joint_friction="${joint_1_friction}" joint_lower_limit="${joint_1_lower_limit}" joint_upper_limit="${joint_1_upper_limit}" joint_velocity_limit="${joint_1_velocity_limit}" joint_torque_limit="${joint_1_torque_limit}" safety_limits="${safety_limits}" safety_position_margin="${safety_position_margin}" safety_k_position="${safety_k_position}"/>
+    <xacro:kinova_armjoint joint_name="${prefix}joint_1" type="${joint_1_type}" parent="${prefix}link_base" child="${prefix}link_1" joint_axis_xyz="${joint_1_axis_xyz}" joint_origin_xyz="${joint_1_origin_xyz}" joint_origin_rpy="${joint_1_origin_rpy}" joint_damping="${joint_1_damping}" joint_friction="${joint_1_friction}" joint_lower_limit="${joint_1_lower_limit}" joint_upper_limit="${joint_1_upper_limit}" joint_velocity_limit="${joint_1_velocity_limit}" joint_torque_limit="${joint_1_torque_limit}" safety_limits="${safety_limits}" safety_position_margin="${safety_position_margin}" safety_k_position="${safety_k_position}" gazebo_preserve_fixed_joint="${gazebo_preserve_fixed_joint}"/>
     <xacro:kinova_armlink link_name="${prefix}link_2" link_mesh="${link_2_mesh}" use_ring_mesh="true" mu="${link_2_mu}"/>
-    <xacro:kinova_armjoint joint_name="${prefix}joint_2" type="${joint_2_type}" parent="${prefix}link_1" child="${prefix}link_2" joint_axis_xyz="${joint_2_axis_xyz}" joint_origin_xyz="${joint_2_origin_xyz}" joint_origin_rpy="${joint_2_origin_rpy}" joint_damping="${joint_2_damping}" joint_friction="${joint_2_friction}" joint_lower_limit="${joint_2_lower_limit}" joint_upper_limit="${joint_2_upper_limit}" joint_velocity_limit="${joint_2_velocity_limit}" joint_torque_limit="${joint_2_torque_limit}" safety_limits="${safety_limits}" safety_position_margin="${safety_position_margin}" safety_k_position="${safety_k_position}"/>
+    <xacro:kinova_armjoint joint_name="${prefix}joint_2" type="${joint_2_type}" parent="${prefix}link_1" child="${prefix}link_2" joint_axis_xyz="${joint_2_axis_xyz}" joint_origin_xyz="${joint_2_origin_xyz}" joint_origin_rpy="${joint_2_origin_rpy}" joint_damping="${joint_2_damping}" joint_friction="${joint_2_friction}" joint_lower_limit="${joint_2_lower_limit}" joint_upper_limit="${joint_2_upper_limit}" joint_velocity_limit="${joint_2_velocity_limit}" joint_torque_limit="${joint_2_torque_limit}" safety_limits="${safety_limits}" safety_position_margin="${safety_position_margin}" safety_k_position="${safety_k_position}" gazebo_preserve_fixed_joint="${gazebo_preserve_fixed_joint}"/>
     <xacro:kinova_armlink link_name="${prefix}link_3" link_mesh="${link_3_mesh}" use_ring_mesh="true" mu="${link_3_mu}"/>
-    <xacro:kinova_armjoint joint_name="${prefix}joint_3" type="${joint_3_type}" parent="${prefix}link_2" child="${prefix}link_3" joint_axis_xyz="${joint_3_axis_xyz}" joint_origin_xyz="${joint_3_origin_xyz}" joint_origin_rpy="${joint_3_origin_rpy}" joint_damping="${joint_3_damping}" joint_friction="${joint_3_friction}" joint_lower_limit="${joint_3_lower_limit}" joint_upper_limit="${joint_3_upper_limit}" joint_velocity_limit="${joint_3_velocity_limit}" joint_torque_limit="${joint_3_torque_limit}" safety_limits="${safety_limits}" safety_position_margin="${safety_position_margin}" safety_k_position="${safety_k_position}"/>
+    <xacro:kinova_armjoint joint_name="${prefix}joint_3" type="${joint_3_type}" parent="${prefix}link_2" child="${prefix}link_3" joint_axis_xyz="${joint_3_axis_xyz}" joint_origin_xyz="${joint_3_origin_xyz}" joint_origin_rpy="${joint_3_origin_rpy}" joint_damping="${joint_3_damping}" joint_friction="${joint_3_friction}" joint_lower_limit="${joint_3_lower_limit}" joint_upper_limit="${joint_3_upper_limit}" joint_velocity_limit="${joint_3_velocity_limit}" joint_torque_limit="${joint_3_torque_limit}" safety_limits="${safety_limits}" safety_position_margin="${safety_position_margin}" safety_k_position="${safety_k_position}" gazebo_preserve_fixed_joint="${gazebo_preserve_fixed_joint}"/>
     <xacro:kinova_armlink link_name="${prefix}link_4" link_mesh="${link_4_mesh}" use_ring_mesh="true" mu="${link_4_mu}"/>
-    <xacro:kinova_armjoint joint_name="${prefix}joint_4" type="${joint_4_type}" parent="${prefix}link_3" child="${prefix}link_4" joint_axis_xyz="${joint_4_axis_xyz}" joint_origin_xyz="${joint_4_origin_xyz}" joint_origin_rpy="${joint_4_origin_rpy}" joint_damping="${joint_4_damping}" joint_friction="${joint_4_friction}" joint_lower_limit="${joint_4_lower_limit}" joint_upper_limit="${joint_4_upper_limit}" joint_velocity_limit="${joint_4_velocity_limit}" joint_torque_limit="${joint_4_torque_limit}" safety_limits="${safety_limits}" safety_position_margin="${safety_position_margin}" safety_k_position="${safety_k_position}"/>
+    <xacro:kinova_armjoint joint_name="${prefix}joint_4" type="${joint_4_type}" parent="${prefix}link_3" child="${prefix}link_4" joint_axis_xyz="${joint_4_axis_xyz}" joint_origin_xyz="${joint_4_origin_xyz}" joint_origin_rpy="${joint_4_origin_rpy}" joint_damping="${joint_4_damping}" joint_friction="${joint_4_friction}" joint_lower_limit="${joint_4_lower_limit}" joint_upper_limit="${joint_4_upper_limit}" joint_velocity_limit="${joint_4_velocity_limit}" joint_torque_limit="${joint_4_torque_limit}" safety_limits="${safety_limits}" safety_position_margin="${safety_position_margin}" safety_k_position="${safety_k_position}" gazebo_preserve_fixed_joint="${gazebo_preserve_fixed_joint}"/>
     <xacro:kinova_armlink link_name="${prefix}link_5" link_mesh="${link_5_mesh}" use_ring_mesh="true" ring_mesh="ring_small" mu="${link_5_mu}"/>
-    <xacro:kinova_armjoint joint_name="${prefix}joint_5" type="${joint_5_type}" parent="${prefix}link_4" child="${prefix}link_5" joint_axis_xyz="${joint_5_axis_xyz}" joint_origin_xyz="${joint_5_origin_xyz}" joint_origin_rpy="${joint_5_origin_rpy}" joint_damping="${joint_5_damping}" joint_friction="${joint_5_friction}" joint_lower_limit="${joint_5_lower_limit}" joint_upper_limit="${joint_5_upper_limit}" joint_velocity_limit="${joint_5_velocity_limit}" joint_torque_limit="${joint_5_torque_limit}" safety_limits="${safety_limits}" safety_position_margin="${safety_position_margin}" safety_k_position="${safety_k_position}"/>
+    <xacro:kinova_armjoint joint_name="${prefix}joint_5" type="${joint_5_type}" parent="${prefix}link_4" child="${prefix}link_5" joint_axis_xyz="${joint_5_axis_xyz}" joint_origin_xyz="${joint_5_origin_xyz}" joint_origin_rpy="${joint_5_origin_rpy}" joint_damping="${joint_5_damping}" joint_friction="${joint_5_friction}" joint_lower_limit="${joint_5_lower_limit}" joint_upper_limit="${joint_5_upper_limit}" joint_velocity_limit="${joint_5_velocity_limit}" joint_torque_limit="${joint_5_torque_limit}" safety_limits="${safety_limits}" safety_position_margin="${safety_position_margin}" safety_k_position="${safety_k_position}" gazebo_preserve_fixed_joint="${gazebo_preserve_fixed_joint}"/>
     <xacro:kinova_armlink link_name="${prefix}link_6" link_mesh="${link_6_mesh}" use_ring_mesh="true" ring_mesh="ring_small" mu="${link_6_mu}"/>
-    <xacro:kinova_armjoint joint_name="${prefix}joint_6" type="${joint_6_type}" parent="${prefix}link_5" child="${prefix}link_6" joint_axis_xyz="${joint_6_axis_xyz}" joint_origin_xyz="${joint_6_origin_xyz}" joint_origin_rpy="${joint_6_origin_rpy}" joint_damping="${joint_6_damping}" joint_friction="${joint_6_friction}" joint_lower_limit="${joint_6_lower_limit}" joint_upper_limit="${joint_6_upper_limit}" joint_velocity_limit="${joint_6_velocity_limit}" joint_torque_limit="${joint_6_torque_limit}" safety_limits="${safety_limits}" safety_position_margin="${safety_position_margin}" safety_k_position="${safety_k_position}"/>
+    <xacro:kinova_armjoint joint_name="${prefix}joint_6" type="${joint_6_type}" parent="${prefix}link_5" child="${prefix}link_6" joint_axis_xyz="${joint_6_axis_xyz}" joint_origin_xyz="${joint_6_origin_xyz}" joint_origin_rpy="${joint_6_origin_rpy}" joint_damping="${joint_6_damping}" joint_friction="${joint_6_friction}" joint_lower_limit="${joint_6_lower_limit}" joint_upper_limit="${joint_6_upper_limit}" joint_velocity_limit="${joint_6_velocity_limit}" joint_torque_limit="${joint_6_torque_limit}" safety_limits="${safety_limits}" safety_position_margin="${safety_position_margin}" safety_k_position="${safety_k_position}" gazebo_preserve_fixed_joint="${gazebo_preserve_fixed_joint}"/>
     <xacro:kinova_armlink link_name="${prefix}link_7" link_mesh="${link_7_mesh}" use_ring_mesh="true" ring_mesh="ring_small" mu="${link_7_mu}"/>
-    <xacro:kinova_armjoint joint_name="${prefix}joint_7" type="${joint_7_type}" parent="${prefix}link_6" child="${prefix}link_7" joint_axis_xyz="${joint_7_axis_xyz}" joint_origin_xyz="${joint_7_origin_xyz}" joint_origin_rpy="${joint_7_origin_rpy}" joint_damping="${joint_7_damping}" joint_friction="${joint_7_friction}" joint_lower_limit="${joint_7_lower_limit}" joint_upper_limit="${joint_7_upper_limit}" joint_velocity_limit="${joint_7_velocity_limit}" joint_torque_limit="${joint_7_torque_limit}" safety_limits="${safety_limits}" safety_position_margin="${safety_position_margin}" safety_k_position="${safety_k_position}"/>
-    <xacro:kinova_virtual_fixed_link joint_name="${prefix}joint_end_effector" parent="${prefix}link_7" child="${prefix}end_effector" joint_origin_xyz="${joint_end_effector_origin_xyz}" joint_origin_rpy="${joint_end_effector_origin_rpy}"/>
+    <xacro:kinova_armjoint joint_name="${prefix}joint_7" type="${joint_7_type}" parent="${prefix}link_6" child="${prefix}link_7" joint_axis_xyz="${joint_7_axis_xyz}" joint_origin_xyz="${joint_7_origin_xyz}" joint_origin_rpy="${joint_7_origin_rpy}" joint_damping="${joint_7_damping}" joint_friction="${joint_7_friction}" joint_lower_limit="${joint_7_lower_limit}" joint_upper_limit="${joint_7_upper_limit}" joint_velocity_limit="${joint_7_velocity_limit}" joint_torque_limit="${joint_7_torque_limit}" safety_limits="${safety_limits}" safety_position_margin="${safety_position_margin}" safety_k_position="${safety_k_position}" gazebo_preserve_fixed_joint="${gazebo_preserve_fixed_joint}"/>
+    <xacro:kinova_virtual_fixed_link joint_name="${prefix}joint_end_effector" parent="${prefix}link_7" child="${prefix}end_effector" joint_origin_xyz="${joint_end_effector_origin_xyz}" joint_origin_rpy="${joint_end_effector_origin_rpy}" gazebo_preserve_fixed_joint="${gazebo_preserve_fixed_joint}"/>
     <xacro:kinova_3fingers link_hand="${prefix}link_7" prefix="${prefix}"/>
     <!-- ROS 2 control -->

File: lunalab_summit_xl_gen_description/urdf/manipulators/kinova/kinova_common.xacro (robot description, xacro)
@@ -76,4 +76,5 @@
     safety_position_margin:=${10*pi/180}
     safety_k_position:=20.0
+    gazebo_preserve_fixed_joint:=false
   ">
     <xacro:if value="${(type == 'fixed' and not fixed) or (type != 'fixed' and fixed)}">
@@ -112,4 +113,12 @@
       </xacro:if>
     </joint>
+    <xacro:if value="${fixed}">
+      <xacro:if value="${gazebo_preserve_fixed_joint}">
+        <gazebo reference="${joint_name}">
+          <preserveFixedJoint>true</preserveFixedJoint>
+          <disableFixedJointLumping>true</disableFixedJointLumping>
+        </gazebo>
+      </xacro:if>
+    </xacro:if>
     <xacro:unless value="${fixed}">
       <transmission name="${joint_name}_trans">
@@ -134,6 +143,14 @@
     joint_origin_xyz
     joint_origin_rpy
+    gazebo_preserve_fixed_joint:=false
   ">
-    <link name="${child}"/>
+    <link name="${child}">
+      <xacro:if value="${gazebo_preserve_fixed_joint}">
+        <inertial>
+          <mass value="1e-5"/>
+          <inertia ixx="1e-35" iyy="1e-35" izz="1e-35" ixy="0.0" ixz="0.0" iyz="0.0"/>
+        </inertial>
+      </xacro:if>
+    </link>
     <joint name="${joint_name}" type="fixed">
       <parent link="${parent}"/>
@@ -141,4 +158,10 @@
       <origin xyz="${joint_origin_xyz}" rpy="${joint_origin_rpy}"/>
     </joint>
+    <xacro:if value="${gazebo_preserve_fixed_joint}">
+      <gazebo reference="${joint_name}">
+        <preserveFixedJoint>true</preserveFixedJoint>
+        <disableFixedJointLumping>true</disableFixedJointLumping>
+      </gazebo>
+    </xacro:if>
   </xacro:macro>
 </robot>

File: lunalab_summit_xl_gen_description/urdf/summit_xl/summit_xl.xacro (robot description, xacro)
@@ -28,4 +28,5 @@
     add_base_footprint:=true
     high_quality_mesh:=true
+    gazebo_preserve_fixed_joint:=false
     gazebo_diff_drive:=true
   ">
@@ -33,5 +34,5 @@
     <xacro:property name="wheel_radius" value="${rubber_wheel_radius}"/>
     <!-- Summit XL base -->
-    <xacro:summit_xl_base prefix="${prefix}" add_base_footprint="${add_base_footprint}" high_quality_mesh="${high_quality_mesh}"/>
+    <xacro:summit_xl_base prefix="${prefix}" add_base_footprint="${add_base_footprint}" high_quality_mesh="${high_quality_mesh}" gazebo_preserve_fixed_joint="${gazebo_preserve_fixed_joint}"/>
     <!-- Wheels (rubber) -->
     <xacro:rubber_wheel prefix="${prefix}front_left_" parent="${prefix}base_link" left_wheel="true" high_quality_mesh="${high_quality_mesh}">

File: lunalab_summit_xl_gen_description/urdf/summit_xl/summit_xl_base.xacro (robot description, xacro)
@@ -8,7 +8,15 @@
     add_base_footprint
     high_quality_mesh
+    gazebo_preserve_fixed_joint:=false
   ">
     <xacro:if value="${add_base_footprint}">
-      <link name="${prefix}base_footprint"/>
+      <link name="${prefix}base_footprint">
+        <xacro:if value="${gazebo_preserve_fixed_joint}">
+          <inertial>
+            <mass value="1e-5"/>
+            <inertia ixx="1e-35" iyy="1e-35" izz="1e-35" ixy="0.0" ixz="0.0" iyz="0.0"/>
+          </inertial>
+        </xacro:if>
+      </link>
       <joint name="${prefix}base_footprint_joint" type="fixed">
         <origin xyz="0 0 ${wheel_radius}" rpy="0 0 0"/>
@@ -16,4 +24,10 @@
         <child link="${prefix}base_link"/>
       </joint>
+      <xacro:if value="${gazebo_preserve_fixed_joint}">
+        <gazebo reference="${prefix}base_footprint_joint">
+          <preserveFixedJoint>true</preserveFixedJoint>
+          <disableFixedJointLumping>true</disableFixedJointLumping>
+        </gazebo>
+      </xacro:if>
     </xacro:if>
     <link name="${prefix}base_link">
@@ -36,4 +50,12 @@
       </collision>
     </link>
+    <link name="${prefix}base_docking_contact_link">
+      <xacro:if value="${gazebo_preserve_fixed_joint}">
+        <inertial>
+          <mass value="1e-5"/>
+          <inertia ixx="1e-35" iyy="1e-35" izz="1e-35" ixy="0.0" ixz="0.0" iyz="0.0"/>
+        </inertial>
+      </xacro:if>
+    </link>
     <joint name="${prefix}base_docking_joint" type="fixed">
       <origin xyz="0.284 0.012 0.068" rpy="0 0 0 "/>
@@ -41,5 +63,10 @@
       <child link="${prefix}base_docking_contact_link"/>
     </joint>
-    <link name="${prefix}base_docking_contact_link"/>
+    <xacro:if value="${gazebo_preserve_fixed_joint}">
+      <gazebo reference="${prefix}base_docking_joint">
+        <preserveFixedJoint>true</preserveFixedJoint>
+        <disableFixedJointLumping>true</disableFixedJointLumping>
+      </gazebo>
+    </xacro:if>
   </xacro:macro>
 </robot>
