Commit message: Add xacro args for disabling collision entities
Signed-off-by: Andrej Orsula <orsula.andrej@gmail.com>

File: lunalab_summit_xl_gen_description/urdf/lunalab_summit_xl_gen.urdf.xacro (robot description, xacro)
@@ -28,4 +28,12 @@
   <!-- Parametric k-position factor of all safety controllers -->
   <xacro:arg name="safety_k_position" default="20"/>
+  <!-- Flag to enable collision geometry for the chassis of Summit XL -->
+  <xacro:arg name="collision_chassis" default="true"/>
+  <!-- Flag to enable collision geometry for the wheels fo Summit XL -->
+  <xacro:arg name="collision_wheels" default="true"/>
+  <!-- Flag to enable collision geometry for manipulator's arm -->
+  <xacro:arg name="collision_arm" default="true"/>
+  <!-- Flag to enable collision geometry for manipulator's gripper (hand and fingers) -->
+  <xacro:arg name="collision_gripper" default="true"/>
   <!-- (unimplemented!) Flag to select the high or low quality model -->
   <xacro:arg name="high_quality_mesh" default="ignored"/>
@@ -53,14 +61,11 @@
   <!-- Properties -->
   <!--            -->
-  <!-- Manipulator offset (from base_link to the center of the manipulator's base) -->
-  <xacro:property name="manipulator_offset_x" value="0.204"/>
-  <xacro:property name="manipulator_offset_y" value="0.0"/>
-  <xacro:property name="manipulator_offset_z" value="0.11"/>
-  <xacro:property name="manipulator_offset_r" value="0.0"/>
-  <xacro:property name="manipulator_offset_p" value="0.0"/>
-  <xacro:property name="manipulator_offset_y" value="0.0"/>
   <!-- Prefixes -->
   <xacro:property name="prefix_summit_xl" value="$(arg prefix)summit_xl_"/>
   <xacro:property name="prefix_manipulator" value="$(arg prefix)j2s7s300_"/>
+  <!-- Manipulator offset -->
+  <xacro:property name="manipulator_base_parent" value="${prefix_summit_xl}base_link"/>
+  <xacro:property name="manipulator_offset_xyz" value="0.204 0.0 0.11"/>
+  <xacro:property name="manipulator_offset_rpy" value="0.0 0.0 0.0"/>
   <!--       -->
   <!-- Robot -->
@@ -70,4 +75,6 @@
     prefix="${prefix_summit_xl}"
     add_base_footprint="true"
+    collision_chassis="$(arg collision_chassis)"
+    collision_wheels="$(arg collision_wheels)"
     high_quality_mesh="$(arg high_quality_mesh)"
     ros2_control="$(arg ros2_control)"
@@ -79,11 +86,13 @@
   <!-- Kinova Gen2 (Jaco2, spherical wrist, 7DOF, 3-finger gripper) -->
   <xacro:j2s7s300
-    base_parent="${prefix_summit_xl}base_link"
+    base_parent="${manipulator_base_parent}"
     prefix="${prefix_manipulator}"
-    joint_base_origin_xyz="${manipulator_offset_x} ${manipulator_offset_y} ${manipulator_offset_z}"
-    joint_base_origin_rpy="${manipulator_offset_r} ${manipulator_offset_p} ${manipulator_offset_y}"
+    joint_base_origin_xyz="${manipulator_offset_xyz}"
+    joint_base_origin_rpy="${manipulator_offset_rpy}"
     safety_limits="$(arg safety_limits)"
     safety_position_margin="$(arg safety_position_margin)"
     safety_k_position="$(arg safety_k_position)"
+    collision_arm="$(arg collision_arm)"
+    collision_gripper="$(arg collision_gripper)"
     high_quality_mesh="$(arg high_quality_mesh)"
     mimic_gripper_joints="$(arg mimic_gripper_joints)"

File: lunalab_summit_xl_gen_description/urdf/manipulators/kinova/j2s7s300.xacro (robot description, xacro)
@@ -133,4 +133,6 @@
     safety_k_position:=20.0
     high_quality_mesh:=false
+    collision_arm:=true
+    collision_gripper:=true
     mimic_gripper_joints:=false
     ros2_control:=true
@@ -140,22 +142,22 @@
     gazebo_joint_trajectory_controller:=true
   ">
-    <xacro:kinova_armlink link_name="${prefix}link_base" link_mesh="${link_base_mesh}" mu="${link_base_mu}"/>
+    <xacro:kinova_armlink link_name="${prefix}link_base" link_mesh="${link_base_mesh}" collision="${collision_arm}" mu="${link_base_mu}"/>
     <xacro:kinova_armjoint joint_name="${prefix}joint_base" type="${joint_base_type}" parent="${base_parent}" child="${prefix}link_base" joint_axis_xyz="${joint_base_axis_xyz}" joint_origin_xyz="${joint_base_origin_xyz}" joint_origin_rpy="${joint_base_origin_rpy}" joint_lower_limit="0" joint_upper_limit="0" joint_velocity_limit="0" joint_torque_limit="0" fixed="true" safety_limits="${safety_limits}" safety_position_margin="${safety_position_margin}" safety_k_position="${safety_k_position}" gazebo_preserve_fixed_joint="${gazebo_preserve_fixed_joint}"/>
-    <xacro:kinova_armlink link_name="${prefix}link_1" link_mesh="${link_1_mesh}" use_ring_mesh="true" mu="${link_1_mu}"/>
+    <xacro:kinova_armlink link_name="${prefix}link_1" link_mesh="${link_1_mesh}" use_ring_mesh="true" collision="${collision_arm}" mu="${link_1_mu}"/>
     <xacro:kinova_armjoint joint_name="${prefix}joint_1" type="${joint_1_type}" parent="${prefix}link_base" child="${prefix}link_1" joint_axis_xyz="${joint_1_axis_xyz}" joint_origin_xyz="${joint_1_origin_xyz}" joint_origin_rpy="${joint_1_origin_rpy}" joint_damping="${joint_1_damping}" joint_friction="${joint_1_friction}" joint_lower_limit="${joint_1_lower_limit}" joint_upper_limit="${joint_1_upper_limit}" joint_velocity_limit="${joint_1_velocity_limit}" joint_torque_limit="${joint_1_torque_limit}" safety_limits="${safety_limits}" safety_position_margin="${safety_position_margin}" safety_k_position="${safety_k_position}" gazebo_preserve_fixed_joint="${gazebo_preserve_fixed_joint}"/>
-    <xacro:kinova_armlink link_name="${prefix}link_2" link_mesh="${link_2_mesh}" use_ring_mesh="true" mu="${link_2_mu}"/>
+    <xacro:kinova_armlink link_name="${prefix}link_2" link_mesh="${link_2_mesh}" use_ring_mesh="true" collision="${collision_arm}" mu="${link_2_mu}"/>
     <xacro:kinova_armjoint joint_name="${prefix}joint_2" type="${joint_2_type}" parent="${prefix}link_1" child="${prefix}link_2" joint_axis_xyz="${joint_2_axis_xyz}" joint_origin_xyz="${joint_2_origin_xyz}" joint_origin_rpy="${joint_2_origin_rpy}" joint_damping="${joint_2_damping}" joint_friction="${joint_2_friction}" joint_lower_limit="${joint_2_lower_limit}" joint_upper_limit="${joint_2_upper_limit}" joint_velocity_limit="${joint_2_velocity_limit}" joint_torque_limit="${joint_2_torque_limit}" safety_limits="${safety_limits}" safety_position_margin="${safety_position_margin}" safety_k_position="${safety_k_position}" gazebo_preserve_fixed_joint="${gazebo_preserve_fixed_joint}"/>
-    <xacro:kinova_armlink link_name="${prefix}link_3" link_mesh="${link_3_mesh}" use_ring_mesh="true" mu="${link_3_mu}"/>
+    <xacro:kinova_armlink link_name="${prefix}link_3" link_mesh="${link_3_mesh}" use_ring_mesh="true" collision="${collision_arm}" mu="${link_3_mu}"/>
     <xacro:kinova_armjoint joint_name="${prefix}joint_3" type="${joint_3_type}" parent="${prefix}link_2" child="${prefix}link_3" joint_axis_xyz="${joint_3_axis_xyz}" joint_origin_xyz="${joint_3_origin_xyz}" joint_origin_rpy="${joint_3_origin_rpy}" joint_damping="${joint_3_damping}" joint_friction="${joint_3_friction}" joint_lower_limit="${joint_3_lower_limit}" joint_upper_limit="${joint_3_upper_limit}" joint_velocity_limit="${joint_3_velocity_limit}" joint_torque_limit="${joint_3_torque_limit}" safety_limits="${safety_limits}" safety_position_margin="${safety_position_margin}" safety_k_position="${safety_k_position}" gazebo_preserve_fixed_joint="${gazebo_preserve_fixed_joint}"/>
-    <xacro:kinova_armlink link_name="${prefix}link_4" link_mesh="${link_4_mesh}" use_ring_mesh="true" mu="${link_4_mu}"/>
+    <xacro:kinova_armlink link_name="${prefix}link_4" link_mesh="${link_4_mesh}" use_ring_mesh="true" collision="${collision_arm}" mu="${link_4_mu}"/>
     <xacro:kinova_armjoint joint_name="${prefix}joint_4" type="${joint_4_type}" parent="${prefix}link_3" child="${prefix}link_4" joint_axis_xyz="${joint_4_axis_xyz}" joint_origin_xyz="${joint_4_origin_xyz}" joint_origin_rpy="${joint_4_origin_rpy}" joint_damping="${joint_4_damping}" joint_friction="${joint_4_friction}" joint_lower_limit="${joint_4_lower_limit}" joint_upper_limit="${joint_4_upper_limit}" joint_velocity_limit="${joint_4_velocity_limit}" joint_torque_limit="${joint_4_torque_limit}" safety_limits="${safety_limits}" safety_position_margin="${safety_position_margin}" safety_k_position="${safety_k_position}" gazebo_preserve_fixed_joint="${gazebo_preserve_fixed_joint}"/>
-    <xacro:kinova_armlink link_name="${prefix}link_5" link_mesh="${link_5_mesh}" use_ring_mesh="true" ring_mesh="ring_small" mu="${link_5_mu}"/>
+    <xacro:kinova_armlink link_name="${prefix}link_5" link_mesh="${link_5_mesh}" use_ring_mesh="true" ring_mesh="ring_small" collision="${collision_arm}" mu="${link_5_mu}"/>
     <xacro:kinova_armjoint joint_name="${prefix}joint_5" type="${joint_5_type}" parent="${prefix}link_4" child="${prefix}link_5" joint_axis_xyz="${joint_5_axis_xyz}" joint_origin_xyz="${joint_5_origin_xyz}" joint_origin_rpy="${joint_5_origin_rpy}" joint_damping="${joint_5_damping}" joint_friction="${joint_5_friction}" joint_lower_limit="${joint_5_lower_limit}" joint_upper_limit="${joint_5_upper_limit}" joint_velocity_limit="${joint_5_velocity_limit}" joint_torque_limit="${joint_5_torque_limit}" safety_limits="${safety_limits}" safety_position_margin="${safety_position_margin}" safety_k_position="${safety_k_position}" gazebo_preserve_fixed_joint="${gazebo_preserve_fixed_joint}"/>
-    <xacro:kinova_armlink link_name="${prefix}link_6" link_mesh="${link_6_mesh}" use_ring_mesh="true" ring_mesh="ring_small" mu="${link_6_mu}"/>
+    <xacro:kinova_armlink link_name="${prefix}link_6" link_mesh="${link_6_mesh}" use_ring_mesh="true" ring_mesh="ring_small" collision="${collision_arm}" mu="${link_6_mu}"/>
     <xacro:kinova_armjoint joint_name="${prefix}joint_6" type="${joint_6_type}" parent="${prefix}link_5" child="${prefix}link_6" joint_axis_xyz="${joint_6_axis_xyz}" joint_origin_xyz="${joint_6_origin_xyz}" joint_origin_rpy="${joint_6_origin_rpy}" joint_damping="${joint_6_damping}" joint_friction="${joint_6_friction}" joint_lower_limit="${joint_6_lower_limit}" joint_upper_limit="${joint_6_upper_limit}" joint_velocity_limit="${joint_6_velocity_limit}" joint_torque_limit="${joint_6_torque_limit}" safety_limits="${safety_limits}" safety_position_margin="${safety_position_margin}" safety_k_position="${safety_k_position}" gazebo_preserve_fixed_joint="${gazebo_preserve_fixed_joint}"/>
-    <xacro:kinova_armlink link_name="${prefix}link_7" link_mesh="${link_7_mesh}" use_ring_mesh="true" ring_mesh="ring_small" mu="${link_7_mu}"/>
+    <xacro:kinova_armlink link_name="${prefix}link_7" link_mesh="${link_7_mesh}" use_ring_mesh="true" ring_mesh="ring_small" collision="${collision_gripper}" mu="${link_7_mu}"/>
     <xacro:kinova_armjoint joint_name="${prefix}joint_7" type="${joint_7_type}" parent="${prefix}link_6" child="${prefix}link_7" joint_axis_xyz="${joint_7_axis_xyz}" joint_origin_xyz="${joint_7_origin_xyz}" joint_origin_rpy="${joint_7_origin_rpy}" joint_damping="${joint_7_damping}" joint_friction="${joint_7_friction}" joint_lower_limit="${joint_7_lower_limit}" joint_upper_limit="${joint_7_upper_limit}" joint_velocity_limit="${joint_7_velocity_limit}" joint_torque_limit="${joint_7_torque_limit}" safety_limits="${safety_limits}" safety_position_margin="${safety_position_margin}" safety_k_position="${safety_k_position}" gazebo_preserve_fixed_joint="${gazebo_preserve_fixed_joint}"/>
     <xacro:kinova_virtual_fixed_link joint_name="${prefix}joint_end_effector" parent="${prefix}link_7" child="${prefix}end_effector" joint_origin_xyz="${joint_end_effector_origin_xyz}" joint_origin_rpy="${joint_end_effector_origin_rpy}" gazebo_preserve_fixed_joint="${gazebo_preserve_fixed_joint}"/>
-    <xacro:kinova_3fingers link_hand="${prefix}link_7" prefix="${prefix}" mimic_joints="${mimic_gripper_joints}"/>
+    <xacro:kinova_3fingers link_hand="${prefix}link_7" prefix="${prefix}" collision="${collision_gripper}" mimic_joints="${mimic_gripper_joints}"/>
     <!-- ROS 2 control -->
     <xacro:if value="${ros2_control}">

File: lunalab_summit_xl_gen_description/urdf/manipulators/kinova/kinova_common.xacro (robot description, xacro)
@@ -13,4 +13,6 @@
   <!-- use_ring_mesh - Flag to enable ring mesh (visual only) -->
   <!-- ring_mesh     - Selector of ring mesh type, which must correspond to mesh name, e.g. `ring_small` -->
+  <!-- collision     - Flag to enable collision geometry -->
+  <!-- mu            - Friction of the surface applied to both directions -->
   <xacro:macro name="kinova_armlink" params="
     link_name
@@ -18,4 +20,5 @@
     use_ring_mesh:=false
     ring_mesh:=ring_big
+    collision:=true
     mu:=1.0
   ">
@@ -34,9 +37,11 @@
         </visual>
       </xacro:if>
-      <collision>
-        <geometry>
-          <mesh filename="package://lunalab_summit_xl_gen_description/meshes/kinova/collision/${link_mesh}.stl"/>
-        </geometry>
-      </collision>
+      <xacro:if value="${collision}">
+        <collision>
+          <geometry>
+            <mesh filename="package://lunalab_summit_xl_gen_description/meshes/kinova/collision/${link_mesh}.stl"/>
+          </geometry>
+        </collision>
+      </xacro:if>
       <xacro:kinova_inertial link_mesh="${link_mesh}"/>
     </link>

File: lunalab_summit_xl_gen_description/urdf/manipulators/kinova/kinova_finger_set.xacro (robot description, xacro)
@@ -48,9 +48,10 @@
     link_hand
     prefix
+    collision:=true
     mimic_joints:=false
   ">
-    <xacro:kinova_finger prefix="${prefix}" finger_number="1" hand="${link_hand}" finger_origin_xyz="${finger_1_of_3_origin_xyz}" finger_origin_rpy="${finger_1_of_3_origin_rpy}" mimic_joints="${mimic_joints}"/>
-    <xacro:kinova_finger prefix="${prefix}" finger_number="2" hand="${link_hand}" finger_origin_xyz="${finger_2_of_3_origin_xyz}" finger_origin_rpy="${finger_2_of_3_origin_rpy}" mimic_joints="${mimic_joints}"/>
-    <xacro:kinova_finger prefix="${prefix}" finger_number="3" hand="${link_hand}" finger_origin_xyz="${finger_3_of_3_origin_xyz}" finger_origin_rpy="${finger_3_of_3_origin_rpy}" mimic_joints="${mimic_joints}"/>
+    <xacro:kinova_finger prefix="${prefix}" finger_number="1" hand="${link_hand}" finger_origin_xyz="${finger_1_of_3_origin_xyz}" finger_origin_rpy="${finger_1_of_3_origin_rpy}" collision="${collision}" mimic_joints="${mimic_joints}"/>
+    <xacro:kinova_finger prefix="${prefix}" finger_number="2" hand="${link_hand}" finger_origin_xyz="${finger_2_of_3_origin_xyz}" finger_origin_rpy="${finger_2_of_3_origin_rpy}" collision="${collision}" mimic_joints="${mimic_joints}"/>
+    <xacro:kinova_finger prefix="${prefix}" finger_number="3" hand="${link_hand}" finger_origin_xyz="${finger_3_of_3_origin_xyz}" finger_origin_rpy="${finger_3_of_3_origin_rpy}" collision="${collision}" mimic_joints="${mimic_joints}"/>
   </xacro:macro>
   <!--       -->
@@ -61,7 +62,8 @@
     prefix
     mimic_joints:=false
+    collision:=true
   ">
-    <xacro:kinova_finger prefix="${prefix}" finger_number="1" hand="${link_hand}" finger_origin_xyz="${finger_1_of_2_origin_xyz}" finger_origin_rpy="${finger_1_of_2_origin_rpy}" mimic_joints="${mimic_joints}"/>
-    <xacro:kinova_finger prefix="${prefix}" finger_number="2" hand="${link_hand}" finger_origin_xyz="${finger_2_of_2_origin_xyz}" finger_origin_rpy="${finger_2_of_2_origin_rpy}" mimic_joints="${mimic_joints}"/>
+    <xacro:kinova_finger prefix="${prefix}" finger_number="1" hand="${link_hand}" finger_origin_xyz="${finger_1_of_2_origin_xyz}" finger_origin_rpy="${finger_1_of_2_origin_rpy}" collision="${collision}" mimic_joints="${mimic_joints}"/>
+    <xacro:kinova_finger prefix="${prefix}" finger_number="2" hand="${link_hand}" finger_origin_xyz="${finger_2_of_2_origin_xyz}" finger_origin_rpy="${finger_2_of_2_origin_rpy}" collision="${collision}" mimic_joints="${mimic_joints}"/>
   </xacro:macro>
   <!--       -->
@@ -74,7 +76,8 @@
     finger_origin_xyz
     finger_origin_rpy
+    collision:=true
     mimic_joints:=false
   ">
-    <xacro:kinova_armlink link_name="${prefix}link_finger_${finger_number}" link_mesh="${finger_proximal_mesh}" mu="${finger_link_proximal_mu}"/>
+    <xacro:kinova_armlink link_name="${prefix}link_finger_${finger_number}" link_mesh="${finger_proximal_mesh}" collision="${collision}" mu="${finger_link_proximal_mu}"/>
     <joint name="${prefix}joint_finger_${finger_number}" type="revolute">
       <parent link="${hand}"/>
@@ -100,5 +103,5 @@
       </actuator>
     </transmission>
-    <xacro:kinova_armlink link_name="${prefix}link_finger_tip_${finger_number}" link_mesh="${finger_distal_mesh}" mu="${finger_link_distal_mu}"/>
+    <xacro:kinova_armlink link_name="${prefix}link_finger_tip_${finger_number}" link_mesh="${finger_distal_mesh}" collision="${collision}" mu="${finger_link_distal_mu}"/>
     <joint name="${prefix}joint_finger_tip_${finger_number}" type="revolute">
       <parent link="${prefix}link_finger_${finger_number}"/>

File: lunalab_summit_xl_gen_description/urdf/summit_xl/rubber_wheel.xacro (robot description, xacro)
@@ -42,4 +42,5 @@
     *origin
     left_wheel
+    collision:=true
     high_quality_mesh
   ">
@@ -64,10 +65,12 @@
         </geometry>
       </visual>
-      <collision>
-        <origin xyz="0 0 0" rpy="${pi/2} 0 0"/>
-        <geometry>
-          <cylinder length="${rubber_wheel_width}" radius="${rubber_wheel_radius}"/>
-        </geometry>
-      </collision>
+      <xacro:if value="${collision}">
+        <collision>
+          <origin xyz="0 0 0" rpy="${pi/2} 0 0"/>
+          <geometry>
+            <cylinder length="${rubber_wheel_width}" radius="${rubber_wheel_radius}"/>
+          </geometry>
+        </collision>
+      </xacro:if>
       <inertial>
         <mass value="${rubber_wheel_mass}"/>

File: lunalab_summit_xl_gen_description/urdf/summit_xl/summit_xl.xacro (robot description, xacro)
@@ -25,4 +25,6 @@
     prefix:=summit_xl_
     add_base_footprint:=true
+    collision_chassis:=true
+    collision_wheels:=true
     high_quality_mesh:=true
     ros2_control:=true
@@ -35,16 +37,16 @@
     <xacro:property name="wheel_radius" value="${rubber_wheel_radius}"/>
     <!-- Summit XL base -->
-    <xacro:summit_xl_base prefix="${prefix}" add_base_footprint="${add_base_footprint}" high_quality_mesh="${high_quality_mesh}" gazebo_preserve_fixed_joint="${gazebo_preserve_fixed_joint}"/>
+    <xacro:summit_xl_base prefix="${prefix}" add_base_footprint="${add_base_footprint}" collision="${collision_chassis}" high_quality_mesh="${high_quality_mesh}" gazebo_preserve_fixed_joint="${gazebo_preserve_fixed_joint}"/>
     <!-- Wheels (rubber) -->
-    <xacro:rubber_wheel prefix="${prefix}front_left_" parent="${prefix}base_link" left_wheel="true" high_quality_mesh="${high_quality_mesh}">
+    <xacro:rubber_wheel prefix="${prefix}front_left_" parent="${prefix}base_link" left_wheel="true" collision="${collision_wheels}" high_quality_mesh="${high_quality_mesh}">
       <origin xyz="${wheel_offset_x} ${wheel_offset_y} ${wheel_offset_z}" rpy="0 0 0"/>
     </xacro:rubber_wheel>
-    <xacro:rubber_wheel prefix="${prefix}back_left_" parent="${prefix}base_link" left_wheel="true" high_quality_mesh="${high_quality_mesh}">
+    <xacro:rubber_wheel prefix="${prefix}back_left_" parent="${prefix}base_link" left_wheel="true" collision="${collision_wheels}" high_quality_mesh="${high_quality_mesh}">
       <origin xyz="-${wheel_offset_x} ${wheel_offset_y} ${wheel_offset_z}" rpy="0 0 0"/>
     </xacro:rubber_wheel>
-    <xacro:rubber_wheel prefix="${prefix}front_right_" parent="${prefix}base_link" left_wheel="false" high_quality_mesh="${high_quality_mesh}">
+    <xacro:rubber_wheel prefix="${prefix}front_right_" parent="${prefix}base_link" left_wheel="false" collision="${collision_wheels}" high_quality_mesh="${high_quality_mesh}">
       <origin xyz="${wheel_offset_x} -${wheel_offset_y} ${wheel_offset_z}" rpy="0 0 0"/>
     </xacro:rubber_wheel>
-    <xacro:rubber_wheel prefix="${prefix}back_right_" parent="${prefix}base_link" left_wheel="false" high_quality_mesh="${high_quality_mesh}">
+    <xacro:rubber_wheel prefix="${prefix}back_right_" parent="${prefix}base_link" left_wheel="false" collision="${collision_wheels}" high_quality_mesh="${high_quality_mesh}">
       <origin xyz="-${wheel_offset_x} -${wheel_offset_y} ${wheel_offset_z}" rpy="0 0 0"/>
     </xacro:rubber_wheel>

File: lunalab_summit_xl_gen_description/urdf/summit_xl/summit_xl_base.xacro (robot description, xacro)
@@ -7,4 +7,5 @@
     prefix
     add_base_footprint
+    collision:=true
     high_quality_mesh
     gazebo_preserve_fixed_joint:=false
@@ -43,10 +44,12 @@
         </geometry>
       </visual>
-      <collision>
-        <origin xyz="0 0 0" rpy="0 0 0 "/>
-        <geometry>
-          <mesh filename="package://lunalab_summit_xl_gen_description/meshes/summit_xl/collision/summit_xl_chassis.stl"/>
-        </geometry>
-      </collision>
+      <xacro:if value="${collision}">
+        <collision>
+          <origin xyz="0 0 0" rpy="0 0 0 "/>
+          <geometry>
+            <mesh filename="package://lunalab_summit_xl_gen_description/meshes/summit_xl/collision/summit_xl_chassis.stl"/>
+          </geometry>
+        </collision>
+      </xacro:if>
     </link>
     <link name="${prefix}base_docking_contact_link">
