Commit message: Integrate with ign_ros2_control
Signed-off-by: Andrej Orsula <orsula.andrej@gmail.com>

File: lunalab_summit_xl_gen_description/urdf/lunalab_summit_xl_gen.urdf (robot description, URDF)
Before this commit: robot lunalab_summit_xl_gen, 22 links, 21 joints
Joints:
- joint robot_j2s7s300_joint_finger_3: origin xyz=-0.02226 -0.02707 -0.11482 rpy=-1.5707963267948966 0.6492624817418906 -1.3861404919338964 -> xyz=-0.02226 -0.02707 -0.11482 rpy=-1.5707963267948966 0.6492624817418906 -1.7554521616558967

File: lunalab_summit_xl_gen_description/urdf/lunalab_summit_xl_gen.urdf.xacro (robot description, xacro)
@@ -30,6 +30,14 @@
   <!-- (unimplemented!) Flag to select the high or low quality model -->
   <xacro:arg name="high_quality_mesh" default="ignored"/>
+  <!-- Flag to mimic joints of the gripper -->
+  <xacro:arg name="mimic_gripper_joints" default="false"/>
   <!-- Flag to enable ros2 controllers for manipulator -->
   <xacro:arg name="ros2_control" default="true"/>
+  <!-- The ros2_control plugin that should be loaded for the manipulator ('fake', 'ignition', 'real' or custom) -->
+  <xacro:arg name="ros2_control_plugin" default="ignition"/>
+  <!-- The output control command interface provided by ros2_control ('position', 'velocity' or 'effort') -->
+  <xacro:arg name="ros2_control_command_interface" default="effort"/>
+  <!-- The filepath to parameters of ROS 2 controllers -->
+  <xacro:arg name="ros2_controller_parameters" default="$(find lunalab_summit_xl_gen_moveit_config)/config/controllers_$(arg ros2_control_command_interface).yaml"/>
   <!-- Flag to preserve fixed joints and prevent lumping when generating SDF for Gazebo -->
   <xacro:arg name="gazebo_preserve_fixed_joint" default="false"/>
@@ -37,7 +45,7 @@
   <xacro:arg name="gazebo_diff_drive" default="true"/>
   <!-- Flag to enable JointTrajectoryController Gazebo plugin for manipulator -->
-  <xacro:arg name="gazebo_joint_trajectory_controller" default="true"/>
+  <xacro:arg name="gazebo_joint_trajectory_controller" default="false"/>
   <!-- Flag to enable JointStatePublisher Gazebo plugin for all joints -->
-  <xacro:arg name="gazebo_joint_state_publisher" default="true"/>
+  <xacro:arg name="gazebo_joint_state_publisher" default="false"/>
   <!-- Flag to enable PosePublisher Gazebo plugin for true pose of robot -->
   <xacro:arg name="gazebo_pose_publisher" default="true"/>
@@ -63,4 +71,7 @@
     add_base_footprint="true"
     high_quality_mesh="$(arg high_quality_mesh)"
+    ros2_control="$(arg ros2_control)"
+    ros2_control_plugin="$(arg ros2_control_plugin)"
+    ros2_control_command_interface="none"
     gazebo_preserve_fixed_joint="$(arg gazebo_preserve_fixed_joint)"
     gazebo_diff_drive="$(arg gazebo_diff_drive)"
@@ -76,5 +87,8 @@
     safety_k_position="$(arg safety_k_position)"
     high_quality_mesh="$(arg high_quality_mesh)"
+    mimic_gripper_joints="$(arg mimic_gripper_joints)"
     ros2_control="$(arg ros2_control)"
+    ros2_control_plugin="$(arg ros2_control_plugin)"
+    ros2_control_command_interface="$(arg ros2_control_command_interface)"
     gazebo_preserve_fixed_joint="$(arg gazebo_preserve_fixed_joint)"
     gazebo_joint_trajectory_controller="$(arg gazebo_joint_trajectory_controller)"
@@ -84,4 +98,10 @@
   <!-- Miscellaneous -->
   <!-- <xacro:lunalab_summit_xl_misc prefix="$(arg prefix)"/> -->
+  <!-- Gazebo - ROS 2 control (Ignition) -->
+  <xacro:if value="$(arg ros2_control)">
+    <xacro:if value="${'ignition' in '$(arg ros2_control_plugin)'}">
+      <xacro:ignition_ros2_control controller_parameters="$(arg ros2_controller_parameters)"/>
+    </xacro:if>
+  </xacro:if>
   <!-- Gazebo - Joint state publisher -->
   <xacro:if value="$(arg gazebo_joint_state_publisher)">

File: lunalab_summit_xl_gen_description/urdf/manipulators/kinova/j2s7s300.xacro (robot description, xacro)
@@ -42,6 +42,6 @@
   <xacro:property name="joint_1_velocity_limit" value="${36*pi/180}"/>
   <xacro:property name="joint_1_torque_limit" value="40"/>
-  <xacro:property name="joint_1_damping" value="16.0"/>
-  <xacro:property name="joint_1_friction" value="0.6"/>
+  <xacro:property name="joint_1_damping" value="14.0"/>
+  <xacro:property name="joint_1_friction" value="0.5"/>
   <xacro:property name="joint_2" value="joint_2"/>
   <xacro:property name="joint_2_type" value="revolute"/>
@@ -53,5 +53,5 @@
   <xacro:property name="joint_2_velocity_limit" value="${36*pi/180}"/>
   <xacro:property name="joint_2_torque_limit" value="80"/>
-  <xacro:property name="joint_2_damping" value="8.5"/>
+  <xacro:property name="joint_2_damping" value="12.0"/>
   <xacro:property name="joint_2_friction" value="0.9"/>
   <xacro:property name="joint_3" value="joint_3"/>
@@ -64,6 +64,6 @@
   <xacro:property name="joint_3_velocity_limit" value="${36*pi/180}"/>
   <xacro:property name="joint_3_torque_limit" value="40"/>
-  <xacro:property name="joint_3_damping" value="7.5"/>
-  <xacro:property name="joint_3_friction" value="0.75"/>
+  <xacro:property name="joint_3_damping" value="10.0"/>
+  <xacro:property name="joint_3_friction" value="0.8"/>
   <xacro:property name="joint_4" value="joint_4"/>
   <xacro:property name="joint_4_type" value="revolute"/>
@@ -75,6 +75,6 @@
   <xacro:property name="joint_4_velocity_limit" value="${36*pi/180}"/>
   <xacro:property name="joint_4_torque_limit" value="40"/>
-  <xacro:property name="joint_4_damping" value="6.5"/>
-  <xacro:property name="joint_4_friction" value="0.95"/>
+  <xacro:property name="joint_4_damping" value="7.0"/>
+  <xacro:property name="joint_4_friction" value="0.55"/>
   <xacro:property name="joint_5" value="joint_5"/>
   <xacro:property name="joint_5_type" value="revolute"/>
@@ -86,5 +86,5 @@
   <xacro:property name="joint_5_velocity_limit" value="${48*pi/180}"/>
   <xacro:property name="joint_5_torque_limit" value="20"/>
-  <xacro:property name="joint_5_damping" value="4.5"/>
+  <xacro:property name="joint_5_damping" value="5.5"/>
   <xacro:property name="joint_5_friction" value="0.35"/>
   <xacro:property name="joint_6" value="joint_6"/>
@@ -97,6 +97,6 @@
   <xacro:property name="joint_6_velocity_limit" value="${48*pi/180}"/>
   <xacro:property name="joint_6_torque_limit" value="20"/>
-  <xacro:property name="joint_6_damping" value="4.0"/>
-  <xacro:property name="joint_6_friction" value="0.3"/>
+  <xacro:property name="joint_6_damping" value="4.5"/>
+  <xacro:property name="joint_6_friction" value="0.25"/>
   <xacro:property name="joint_7" value="joint_7"/>
   <xacro:property name="joint_7_type" value="revolute"/>
@@ -108,5 +108,5 @@
   <xacro:property name="joint_7_velocity_limit" value="${48*pi/180}"/>
   <xacro:property name="joint_7_torque_limit" value="20"/>
-  <xacro:property name="joint_7_damping" value="3.5"/>
+  <xacro:property name="joint_7_damping" value="4.0"/>
   <xacro:property name="joint_7_friction" value="0.2"/>
   <xacro:property name="joint_end_effector" value="end_effector_offset"/>
@@ -133,5 +133,8 @@
     safety_k_position:=20.0
     high_quality_mesh:=false
+    mimic_gripper_joints:=false
     ros2_control:=true
+    ros2_control_plugin:=ignition
+    ros2_control_command_interface:=effort
     gazebo_preserve_fixed_joint:=false
     gazebo_joint_trajectory_controller:=true
@@ -154,9 +157,9 @@
     <xacro:kinova_armjoint joint_name="${prefix}joint_7" type="${joint_7_type}" parent="${prefix}link_6" child="${prefix}link_7" joint_axis_xyz="${joint_7_axis_xyz}" joint_origin_xyz="${joint_7_origin_xyz}" joint_origin_rpy="${joint_7_origin_rpy}" joint_damping="${joint_7_damping}" joint_friction="${joint_7_friction}" joint_lower_limit="${joint_7_lower_limit}" joint_upper_limit="${joint_7_upper_limit}" joint_velocity_limit="${joint_7_velocity_limit}" joint_torque_limit="${joint_7_torque_limit}" safety_limits="${safety_limits}" safety_position_margin="${safety_position_margin}" safety_k_position="${safety_k_position}" gazebo_preserve_fixed_joint="${gazebo_preserve_fixed_joint}"/>
     <xacro:kinova_virtual_fixed_link joint_name="${prefix}joint_end_effector" parent="${prefix}link_7" child="${prefix}end_effector" joint_origin_xyz="${joint_end_effector_origin_xyz}" joint_origin_rpy="${joint_end_effector_origin_rpy}" gazebo_preserve_fixed_joint="${gazebo_preserve_fixed_joint}"/>
-    <xacro:kinova_3fingers link_hand="${prefix}link_7" prefix="${prefix}"/>
+    <xacro:kinova_3fingers link_hand="${prefix}link_7" prefix="${prefix}" mimic_joints="${mimic_gripper_joints}"/>
     <!-- ROS 2 control -->
     <xacro:if value="${ros2_control}">
-      <xacro:ros2_control_j2s7s300_arm name="KinovaArmFakeSystem" prefix="${prefix}"/>
-      <xacro:ros2_control_3fingers name="KinovaGripperFakeSystem" prefix="${prefix}"/>
+      <xacro:ros2_control_j2s7s300_arm prefix="${prefix}" plugin="${ros2_control_plugin}" command_interface="${ros2_control_command_interface}"/>
+      <xacro:ros2_control_3fingers prefix="${prefix}" plugin="${ros2_control_plugin}" command_interface="${ros2_control_command_interface}" mimic_joints="${mimic_gripper_joints}"/>
     </xacro:if>
     <!-- Gazebo - Joint trajectory controller -->

File: lunalab_summit_xl_gen_description/urdf/manipulators/kinova/kinova_finger_set.xacro (robot description, xacro)
@@ -26,6 +26,6 @@
   <xacro:property name="finger_proximal_velocity_limit" value="1.0"/>
   <xacro:property name="finger_proximal_torque_limit" value="2.0"/>
-  <xacro:property name="finger_proximal_damping" value="0.5"/>
-  <xacro:property name="finger_proximal_friction" value="0.05"/>
+  <xacro:property name="finger_proximal_damping" value="0.15"/>
+  <xacro:property name="finger_proximal_friction" value="0.01"/>
   <xacro:property name="finger_link_proximal_mu" value="1.6"/>
   <xacro:property name="finger_distal_origin_xyz" value="0.044 -0.003 0"/>
@@ -37,7 +37,7 @@
   <xacro:property name="finger_distal_velocity_limit" value="1.0"/>
   <xacro:property name="finger_distal_torque_limit" value="2.0"/>
-  <xacro:property name="finger_distal_damping" value="0.05"/>
-  <xacro:property name="finger_distal_friction" value="0.01"/>
-  <xacro:property name="finger_distal_spring_stiffness" value="0.2"/>
+  <xacro:property name="finger_distal_damping" value="0.01"/>
+  <xacro:property name="finger_distal_friction" value="0.0005"/>
+  <xacro:property name="finger_distal_spring_stiffness" value="0.5"/>
   <xacro:property name="finger_distal_spring_reference" value="0.0"/>
   <xacro:property name="finger_link_distal_mu" value="1.6"/>
@@ -48,8 +48,9 @@
     link_hand
     prefix
+    mimic_joints:=false
   ">
-    <xacro:kinova_finger prefix="${prefix}" finger_number="1" hand="${link_hand}" finger_origin_xyz="${finger_1_of_3_origin_xyz}" finger_origin_rpy="${finger_1_of_3_origin_rpy}"/>
-    <xacro:kinova_finger prefix="${prefix}" finger_number="2" hand="${link_hand}" finger_origin_xyz="${finger_2_of_3_origin_xyz}" finger_origin_rpy="${finger_2_of_3_origin_rpy}"/>
-    <xacro:kinova_finger prefix="${prefix}" finger_number="3" hand="${link_hand}" finger_origin_xyz="${finger_3_of_3_origin_xyz}" finger_origin_rpy="${finger_2_of_3_origin_rpy}"/>
+    <xacro:kinova_finger prefix="${prefix}" finger_number="1" hand="${link_hand}" finger_origin_xyz="${finger_1_of_3_origin_xyz}" finger_origin_rpy="${finger_1_of_3_origin_rpy}" mimic_joints="${mimic_joints}"/>
+    <xacro:kinova_finger prefix="${prefix}" finger_number="2" hand="${link_hand}" finger_origin_xyz="${finger_2_of_3_origin_xyz}" finger_origin_rpy="${finger_2_of_3_origin_rpy}" mimic_joints="${mimic_joints}"/>
+    <xacro:kinova_finger prefix="${prefix}" finger_number="3" hand="${link_hand}" finger_origin_xyz="${finger_3_of_3_origin_xyz}" finger_origin_rpy="${finger_3_of_3_origin_rpy}" mimic_joints="${mimic_joints}"/>
   </xacro:macro>
   <!--       -->
@@ -59,7 +60,8 @@
     link_hand
     prefix
+    mimic_joints:=false
   ">
-    <xacro:kinova_finger prefix="${prefix}" finger_number="1" hand="${link_hand}" finger_origin_xyz="${finger_1_of_2_origin_xyz}" finger_origin_rpy="${finger_1_of_2_origin_rpy}"/>
-    <xacro:kinova_finger prefix="${prefix}" finger_number="2" hand="${link_hand}" finger_origin_xyz="${finger_2_of_2_origin_xyz}" finger_origin_rpy="${finger_2_of_2_origin_rpy}"/>
+    <xacro:kinova_finger prefix="${prefix}" finger_number="1" hand="${link_hand}" finger_origin_xyz="${finger_1_of_2_origin_xyz}" finger_origin_rpy="${finger_1_of_2_origin_rpy}" mimic_joints="${mimic_joints}"/>
+    <xacro:kinova_finger prefix="${prefix}" finger_number="2" hand="${link_hand}" finger_origin_xyz="${finger_2_of_2_origin_xyz}" finger_origin_rpy="${finger_2_of_2_origin_rpy}" mimic_joints="${mimic_joints}"/>
   </xacro:macro>
   <!--       -->
@@ -72,4 +74,5 @@
     finger_origin_xyz
     finger_origin_rpy
+    mimic_joints:=false
   ">
     <xacro:kinova_armlink link_name="${prefix}link_finger_${finger_number}" link_mesh="${finger_proximal_mesh}" mu="${finger_link_proximal_mu}"/>
@@ -81,4 +84,9 @@
       <limit lower="${finger_proximal_lower_limit}" upper="${finger_proximal_upper_limit}" effort="${finger_proximal_torque_limit}" velocity="${finger_proximal_velocity_limit}"/>
       <dynamics damping="${finger_proximal_damping}" friction="${finger_proximal_friction}"/>
+       <xacro:if value="${mimic_joints}">
+        <xacro:unless value="${finger_number == 1}">
+          <mimic joint="${prefix}joint_finger_1"/>
+        </xacro:unless>
+      </xacro:if>
     </joint>
     <transmission name="${prefix}joint_finger_${finger_number}_trans">

File: lunalab_summit_xl_gen_description/urdf/summit_xl/rubber_wheel.xacro (robot description, xacro)
@@ -81,5 +81,6 @@
         <hardwareInterface>hardware_interface/VelocityJointInterface</hardwareInterface>
       </joint>
-      <actuator name="${prefix}wheel_joint_motor">
+      <actuator name="${prefix}wheel_joint_actuator">
+        <hardwareInterface>hardware_interface/VelocityJointInterface</hardwareInterface>
         <mechanicalReduction>1</mechanicalReduction>
         <motorTorqueConstant>20</motorTorqueConstant>

File: lunalab_summit_xl_gen_description/urdf/summit_xl/summit_xl.xacro (robot description, xacro)
@@ -5,9 +5,7 @@
   <!-- Imported elements -->
   <!--                   -->
-  <!-- Import Summit XL base -->
   <xacro:include filename="$(find lunalab_summit_xl_gen_description)/urdf/summit_xl/summit_xl_base.xacro"/>
-  <!-- Import Summit XL wheels (rubber) -->
   <xacro:include filename="$(find lunalab_summit_xl_gen_description)/urdf/summit_xl/rubber_wheel.xacro"/>
-  <!-- Gazebo plugins -->
+  <xacro:include filename="$(find lunalab_summit_xl_gen_description)/urdf/summit_xl/summit_xl.ros2_control"/>
   <xacro:include filename="$(find lunalab_summit_xl_gen_description)/urdf/summit_xl/summit_xl.gazebo"/>
   <!--            -->
@@ -28,4 +26,7 @@
     add_base_footprint:=true
     high_quality_mesh:=true
+    ros2_control:=true
+    ros2_control_plugin:=ignition
+    ros2_control_command_interface:=none
     gazebo_preserve_fixed_joint:=false
     gazebo_diff_drive:=true
@@ -48,4 +49,8 @@
       <origin xyz="-${wheel_offset_x} -${wheel_offset_y} ${wheel_offset_z}" rpy="0 0 0"/>
     </xacro:rubber_wheel>
+    <!-- ROS 2 control -->
+    <xacro:if value="${ros2_control}">
+      <xacro:ros2_control_summit_xl prefix="${prefix}" plugin="${ros2_control_plugin}" command_interface="${ros2_control_command_interface}"/>
+    </xacro:if>
     <!-- Gazebo - Differential drive -->
     <xacro:if value="${gazebo_diff_drive}">

Commit message: Fix gripper closing - Orientation of 1st finger origin - Joint positions of predefined "close" group_state
Signed-off-by: Andrej Orsula <orsula.andrej@gmail.com>

File: lunalab_summit_xl_gen_description/urdf/lunalab_summit_xl_gen.urdf (robot description, URDF)
Before this commit: robot lunalab_summit_xl_gen, 22 links, 21 joints
Joints:
- joint robot_j2s7s300_joint_finger_1: origin xyz=0.00279 0.03126 -0.11467 rpy=-1.5707963267948966 0.6492624817418906 1.3596114873035827 -> xyz=0.00279 0.03126 -0.11467 rpy=-1.5707963267948966 0.6492624817418906 1.7819811662862104

File: lunalab_summit_xl_gen_description/urdf/manipulators/kinova/kinova_finger_set.xacro (robot description, xacro)
@@ -10,5 +10,5 @@
   <!-- Finger origin for 3-finger hand -->
   <xacro:property name="finger_1_of_3_origin_xyz" value="0.00279 0.03126 -0.11467"/>
-  <xacro:property name="finger_1_of_3_origin_rpy" value="${-pi/2} ${37.2*pi/180} ${77.9*pi/180}"/>
+  <xacro:property name="finger_1_of_3_origin_rpy" value="${-pi/2} ${37.2*pi/180} ${102.1*pi/180}"/>
   <xacro:property name="finger_2_of_3_origin_xyz" value="0.02226 -0.02707 -0.11482"/>
   <xacro:property name="finger_2_of_3_origin_rpy" value="${-pi/2} ${37.2*pi/180} ${-79.42*pi/180}"/>

File: lunalab_summit_xl_gen_moveit_config/srdf/lunalab_summit_xl_gen_j2s7s300.xacro (robot description, xacro)
@@ -50,7 +50,7 @@
     </group_state>
     <group_state name="close" group="gripper">
-      <joint name="${prefix}j2s7s300_joint_finger_1" value="1.2"/>
-      <joint name="${prefix}j2s7s300_joint_finger_2" value="1.2"/>
-      <joint name="${prefix}j2s7s300_joint_finger_3" value="1.2"/>
+      <joint name="${prefix}j2s7s300_joint_finger_1" value="1.3"/>
+      <joint name="${prefix}j2s7s300_joint_finger_2" value="1.3"/>
+      <joint name="${prefix}j2s7s300_joint_finger_3" value="1.3"/>
     </group_state>
     <end_effector name="gripper" parent_link="${prefix}j2s7s300_end_effector" group="gripper" parent_group="arm"/>

Commit message: Fix origin of 1st finger in 3 finger gripper
Signed-off-by: Andrej Orsula <orsula.andrej@gmail.com>

File: lunalab_summit_xl_gen_description/urdf/lunalab_summit_xl_gen.urdf (robot description, URDF)
Before this commit: robot lunalab_summit_xl_gen, 22 links, 21 joints
Joints:
- joint robot_j2s7s300_joint_finger_1: origin xyz=0.00279 0.03126 -0.11467 rpy=-1.5707963267948966 0.6492624817418906 1.7819811662862104 -> xyz=0.002786 0.03126 -0.114668 rpy=-1.704955772138421 0.6492624817418906 1.6728980880365647
- joint robot_j2s7s300_joint_finger_2: origin xyz=0.02226 -0.02707 -0.11482 rpy=-1.5707963267948966 0.6492624817418906 -1.3861404919338964 -> xyz=0.022256 -0.027073 -0.114668 rpy=-1.5707963267948966 0.6492624817418906 -1.3861404919338964
- joint robot_j2s7s300_joint_finger_3: origin xyz=-0.02226 -0.02707 -0.11482 rpy=-1.5707963267948966 0.6492624817418906 -1.7554521616558967 -> xyz=-0.022256 -0.027073 -0.114668 rpy=-1.5707963267948966 0.6492624817418906 -1.7554521616558967

File: lunalab_summit_xl_gen_description/urdf/manipulators/kinova/kinova_finger_set.xacro (robot description, xacro)
@@ -9,9 +9,9 @@
   <!--            -->
   <!-- Finger origin for 3-finger hand -->
-  <xacro:property name="finger_1_of_3_origin_xyz" value="0.00279 0.03126 -0.11467"/>
-  <xacro:property name="finger_1_of_3_origin_rpy" value="${-pi/2} ${37.2*pi/180} ${102.1*pi/180}"/>
-  <xacro:property name="finger_2_of_3_origin_xyz" value="0.02226 -0.02707 -0.11482"/>
+  <xacro:property name="finger_1_of_3_origin_xyz" value="0.002786 0.03126 -0.114668"/>
+  <xacro:property name="finger_1_of_3_origin_rpy" value="${-97.68677*pi/180} ${37.2*pi/180} ${95.85*pi/180}"/>
+  <xacro:property name="finger_2_of_3_origin_xyz" value="0.022256 -0.027073 -0.114668"/>
   <xacro:property name="finger_2_of_3_origin_rpy" value="${-pi/2} ${37.2*pi/180} ${-79.42*pi/180}"/>
-  <xacro:property name="finger_3_of_3_origin_xyz" value="-0.02226 -0.02707 -0.11482"/>
+  <xacro:property name="finger_3_of_3_origin_xyz" value="-0.022256 -0.027073 -0.114668"/>
   <xacro:property name="finger_3_of_3_origin_rpy" value="${-pi/2} ${37.2*pi/180} ${-100.58*pi/180}"/>
   <!-- Finger origin for 2-finger hand -->

Commit message: Fix j2s7s300 joint_2_torque_limit
Signed-off-by: Andrej Orsula <orsula.andrej@gmail.com>

File: lunalab_summit_xl_gen_description/urdf/lunalab_summit_xl_gen.urdf (robot description, URDF)
Before this commit: robot lunalab_summit_xl_gen, 22 links, 21 joints
Joints:
- joint robot_j2s7s300_joint_2: limit lower=0.8203047484373349 upper=5.462880558742252 effort=80 velocity=0.6283185307179586 -> lower=0.8203047484373349 upper=5.462880558742251 effort=40 velocity=0.6283185307179586
- joint robot_j2s7s300_joint_6: limit lower=1.1344640137963142 upper=5.148721293383272 effort=20 velocity=0.8377580409572781 -> lower=1.1344640137963142 upper=5.1487212933832724 effort=20 velocity=0.8377580409572781

File: lunalab_summit_xl_gen_description/urdf/manipulators/kinova/j2s7s300.xacro (robot description, xacro)
@@ -49,8 +49,8 @@
   <xacro:property name="joint_2_origin_xyz" value="0 0.0016 -0.11875"/>
   <xacro:property name="joint_2_origin_rpy" value="-${pi/2} 0 ${pi}"/>
-  <xacro:property name="joint_2_lower_limit" value="${47/180*pi}"/>
-  <xacro:property name="joint_2_upper_limit" value="${313/180*pi}"/>
+  <xacro:property name="joint_2_lower_limit" value="${47*pi/180}"/>
+  <xacro:property name="joint_2_upper_limit" value="${313*pi/180}"/>
   <xacro:property name="joint_2_velocity_limit" value="${36*pi/180}"/>
-  <xacro:property name="joint_2_torque_limit" value="80"/>
+  <xacro:property name="joint_2_torque_limit" value="40"/>
   <xacro:property name="joint_2_damping" value="12.0"/>
   <xacro:property name="joint_2_friction" value="0.9"/>
@@ -71,6 +71,6 @@
   <xacro:property name="joint_4_origin_xyz" value="0 0 -0.205"/>
   <xacro:property name="joint_4_origin_rpy" value="${pi/2} 0 ${pi}"/>
-  <xacro:property name="joint_4_lower_limit" value="${30/180*pi}"/>
-  <xacro:property name="joint_4_upper_limit" value="${330/180*pi}"/>
+  <xacro:property name="joint_4_lower_limit" value="${30*pi/180}"/>
+  <xacro:property name="joint_4_upper_limit" value="${330*pi/180}"/>
   <xacro:property name="joint_4_velocity_limit" value="${36*pi/180}"/>
   <xacro:property name="joint_4_torque_limit" value="40"/>
@@ -93,6 +93,6 @@
   <xacro:property name="joint_6_origin_xyz" value="0 0 -0.10375"/>
   <xacro:property name="joint_6_origin_rpy" value="${pi/2} 0 ${pi}"/>
-  <xacro:property name="joint_6_lower_limit" value="${65/180*pi}"/>
-  <xacro:property name="joint_6_upper_limit" value="${295/180*pi}"/>
+  <xacro:property name="joint_6_lower_limit" value="${65*pi/180}"/>
+  <xacro:property name="joint_6_upper_limit" value="${295*pi/180}"/>
   <xacro:property name="joint_6_velocity_limit" value="${48*pi/180}"/>
   <xacro:property name="joint_6_torque_limit" value="20"/>
