Commit message: Use joint position limits from tech specs
Signed-off-by: Andrej Orsula <orsula.andrej@gmail.com>

File: lunalab_summit_xl_gen_description/urdf/lunalab_summit_xl_gen.urdf (robot description, URDF)
Before this commit: robot lunalab_summit_xl_gen, 22 links, 21 joints
Joints:
- joint robot_j2s7s300_joint_1: limit lower=-6.283185307179586 upper=6.283185307179586 effort=40 velocity=0.6283185307179586 -> lower=-174.04423300887453 upper=174.04423300887453 effort=40 velocity=0.6283185307179586
- joint robot_j2s7s300_joint_3: limit lower=-6.283185307179586 upper=6.283185307179586 effort=40 velocity=0.6283185307179586 -> lower=-174.04423300887453 upper=174.04423300887453 effort=40 velocity=0.6283185307179586
- joint robot_j2s7s300_joint_5: limit lower=-6.283185307179586 upper=6.283185307179586 effort=20 velocity=0.8377580409572781 -> lower=-174.04423300887453 upper=174.04423300887453 effort=20 velocity=0.8377580409572781
- joint robot_j2s7s300_joint_7: limit lower=-6.283185307179586 upper=6.283185307179586 effort=20 velocity=0.8377580409572781 -> lower=-174.04423300887453 upper=174.04423300887453 effort=20 velocity=0.8377580409572781

File: lunalab_summit_xl_gen_description/urdf/manipulators/kinova/j2s7s300.xacro (robot description, xacro)
@@ -38,6 +38,6 @@
   <xacro:property name="joint_1_origin_xyz" value="0 0 0.15675"/>
   <xacro:property name="joint_1_origin_rpy" value="0 ${pi} 0"/>
-  <xacro:property name="joint_1_lower_limit" value="${-2*pi}"/>
-  <xacro:property name="joint_1_upper_limit" value="${2*pi}"/>
+  <xacro:property name="joint_1_lower_limit" value="${-55.4*pi}"/>
+  <xacro:property name="joint_1_upper_limit" value="${55.4*pi}"/>
   <xacro:property name="joint_1_velocity_limit" value="${36*pi/180}"/>
   <xacro:property name="joint_1_torque_limit" value="40"/>
@@ -60,6 +60,6 @@
   <xacro:property name="joint_3_origin_xyz" value="0 -0.205 0"/>
   <xacro:property name="joint_3_origin_rpy" value="-${pi/2} 0 0"/>
-  <xacro:property name="joint_3_lower_limit" value="${-2*pi}"/>
-  <xacro:property name="joint_3_upper_limit" value="${2*pi}"/>
+  <xacro:property name="joint_3_lower_limit" value="${-55.4*pi}"/>
+  <xacro:property name="joint_3_upper_limit" value="${55.4*pi}"/>
   <xacro:property name="joint_3_velocity_limit" value="${36*pi/180}"/>
   <xacro:property name="joint_3_torque_limit" value="40"/>
@@ -82,6 +82,6 @@
   <xacro:property name="joint_5_origin_xyz" value="0 0.2073 -0.0114"/>
   <xacro:property name="joint_5_origin_rpy" value="${-pi/2} 0 ${pi}"/>
-  <xacro:property name="joint_5_lower_limit" value="${-2*pi}"/>
-  <xacro:property name="joint_5_upper_limit" value="${2*pi}"/>
+  <xacro:property name="joint_5_lower_limit" value="${-55.4*pi}"/>
+  <xacro:property name="joint_5_upper_limit" value="${55.4*pi}"/>
   <xacro:property name="joint_5_velocity_limit" value="${48*pi/180}"/>
   <xacro:property name="joint_5_torque_limit" value="20"/>
@@ -104,6 +104,6 @@
   <xacro:property name="joint_7_origin_xyz" value="0 0.10375 0"/>
   <xacro:property name="joint_7_origin_rpy" value="${-pi/2} 0 ${pi}"/>
-  <xacro:property name="joint_7_lower_limit" value="${-2*pi}"/>
-  <xacro:property name="joint_7_upper_limit" value="${2*pi}"/>
+  <xacro:property name="joint_7_lower_limit" value="${-55.4*pi}"/>
+  <xacro:property name="joint_7_upper_limit" value="${55.4*pi}"/>
   <xacro:property name="joint_7_velocity_limit" value="${48*pi/180}"/>
   <xacro:property name="joint_7_torque_limit" value="20"/>

Commit message: Update default configuration for both sim and real
Signed-off-by: Andrej Orsula <orsula.andrej@gmail.com>

File: lunalab_summit_xl_gen_description/urdf/lunalab_summit_xl_gen.urdf (robot description, URDF)
Before this commit: robot lunalab_summit_xl_gen, 22 links, 21 joints
Joints:
- joint robot_j2s7s300_joint_finger_1: limit lower=0.0 upper=1.51 effort=2.0 velocity=1.0 -> lower=0.0 upper=1.51 effort=5.0 velocity=1.0
- joint robot_j2s7s300_joint_finger_2: limit lower=0.0 upper=1.51 effort=2.0 velocity=1.0 -> lower=0.0 upper=1.51 effort=5.0 velocity=1.0
- joint robot_j2s7s300_joint_finger_3: limit lower=0.0 upper=1.51 effort=2.0 velocity=1.0 -> lower=0.0 upper=1.51 effort=5.0 velocity=1.0

File: lunalab_summit_xl_gen_description/urdf/manipulators/kinova/j2s7s300.xacro (robot description, xacro)
@@ -42,5 +42,5 @@
   <xacro:property name="joint_1_velocity_limit" value="${36*pi/180}"/>
   <xacro:property name="joint_1_torque_limit" value="40"/>
-  <xacro:property name="joint_1_damping" value="14.0"/>
+  <xacro:property name="joint_1_damping" value="15.0"/>
   <xacro:property name="joint_1_friction" value="0.5"/>
   <xacro:property name="joint_2" value="joint_2"/>
@@ -53,5 +53,5 @@
   <xacro:property name="joint_2_velocity_limit" value="${36*pi/180}"/>
   <xacro:property name="joint_2_torque_limit" value="40"/>
-  <xacro:property name="joint_2_damping" value="12.0"/>
+  <xacro:property name="joint_2_damping" value="16.0"/>
   <xacro:property name="joint_2_friction" value="0.9"/>
   <xacro:property name="joint_3" value="joint_3"/>
@@ -64,5 +64,5 @@
   <xacro:property name="joint_3_velocity_limit" value="${36*pi/180}"/>
   <xacro:property name="joint_3_torque_limit" value="40"/>
-  <xacro:property name="joint_3_damping" value="10.0"/>
+  <xacro:property name="joint_3_damping" value="12.0"/>
   <xacro:property name="joint_3_friction" value="0.8"/>
   <xacro:property name="joint_4" value="joint_4"/>
@@ -75,5 +75,5 @@
   <xacro:property name="joint_4_velocity_limit" value="${36*pi/180}"/>
   <xacro:property name="joint_4_torque_limit" value="40"/>
-  <xacro:property name="joint_4_damping" value="7.0"/>
+  <xacro:property name="joint_4_damping" value="8.0"/>
   <xacro:property name="joint_4_friction" value="0.55"/>
   <xacro:property name="joint_5" value="joint_5"/>
@@ -86,5 +86,5 @@
   <xacro:property name="joint_5_velocity_limit" value="${48*pi/180}"/>
   <xacro:property name="joint_5_torque_limit" value="20"/>
-  <xacro:property name="joint_5_damping" value="5.5"/>
+  <xacro:property name="joint_5_damping" value="6.5"/>
   <xacro:property name="joint_5_friction" value="0.35"/>
   <xacro:property name="joint_6" value="joint_6"/>
@@ -97,5 +97,5 @@
   <xacro:property name="joint_6_velocity_limit" value="${48*pi/180}"/>
   <xacro:property name="joint_6_torque_limit" value="20"/>
-  <xacro:property name="joint_6_damping" value="4.5"/>
+  <xacro:property name="joint_6_damping" value="5.5"/>
   <xacro:property name="joint_6_friction" value="0.25"/>
   <xacro:property name="joint_7" value="joint_7"/>
@@ -108,5 +108,5 @@
   <xacro:property name="joint_7_velocity_limit" value="${48*pi/180}"/>
   <xacro:property name="joint_7_torque_limit" value="20"/>
-  <xacro:property name="joint_7_damping" value="4.0"/>
+  <xacro:property name="joint_7_damping" value="4.5"/>
   <xacro:property name="joint_7_friction" value="0.2"/>
   <xacro:property name="joint_end_effector" value="end_effector_offset"/>

File: lunalab_summit_xl_gen_description/urdf/manipulators/kinova/kinova_finger_set.xacro (robot description, xacro)
@@ -25,6 +25,6 @@
   <xacro:property name="finger_proximal_upper_limit" value="1.51"/>
   <xacro:property name="finger_proximal_velocity_limit" value="1.0"/>
-  <xacro:property name="finger_proximal_torque_limit" value="2.0"/>
-  <xacro:property name="finger_proximal_damping" value="0.15"/>
+  <xacro:property name="finger_proximal_torque_limit" value="5.0"/>
+  <xacro:property name="finger_proximal_damping" value="0.3"/>
   <xacro:property name="finger_proximal_friction" value="0.01"/>
   <xacro:property name="finger_link_proximal_mu" value="1.6"/>
@@ -37,7 +37,7 @@
   <xacro:property name="finger_distal_velocity_limit" value="1.0"/>
   <xacro:property name="finger_distal_torque_limit" value="2.0"/>
-  <xacro:property name="finger_distal_damping" value="0.01"/>
-  <xacro:property name="finger_distal_friction" value="0.0005"/>
-  <xacro:property name="finger_distal_spring_stiffness" value="0.5"/>
+  <xacro:property name="finger_distal_damping" value="0.005"/>
+  <xacro:property name="finger_distal_friction" value="0.00025"/>
+  <xacro:property name="finger_distal_spring_stiffness" value="1.25"/>
   <xacro:property name="finger_distal_spring_reference" value="0.0"/>
   <xacro:property name="finger_link_distal_mu" value="1.6"/>

Commit message: Add PBR textures to Summit XL base and Kinova arm
Signed-off-by: Andrej Orsula <orsula.andrej@gmail.com>

File: lunalab_summit_xl_gen_description/urdf/lunalab_summit_xl_gen.urdf (robot description, URDF)
Before this commit: robot lunalab_summit_xl_gen, 22 links, 21 joints
Links:
- link robot_j2s7s300_link_1: geometry collision mesh filename=package://lunalab_summit_xl_gen_description/meshes/kinova/c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; visual mesh filename=package://lunalab_summit_xl_gen_description/meshes/kinova/v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
- link robot_j2s7s300_link_2: geometry collision mesh filename=package://lunalab_summit_xl_gen_description/meshes/kinova/c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; visual mesh filename=package://lunalab_summit_xl_gen_description/meshes/kinova/v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
- link robot_j2s7s300_link_3: geometry collision mesh filename=package://lunalab_summit_xl_gen_description/meshes/kinova/c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; visual mesh filename=package://lunalab_summit_xl_gen_description/meshes/kinova/v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
- link robot_j2s7s300_link_4: geometry collision mesh filename=package://lunalab_summit_xl_gen_description/meshes/kinova/c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; visual mesh filename=package://lunalab_summit_xl_gen_description/meshes/kinova/v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
- link robot_j2s7s300_link_5: geometry collision mesh filename=package://lunalab_summit_xl_gen_description/meshes/kinova/c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; visual mesh filename=package://lunalab_summit_xl_gen_description/meshes/kinova/v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
- link robot_j2s7s300_link_6: geometry collision mesh filename=package://lunalab_summit_xl_gen_description/meshes/kinova/c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; visual mesh filename=package://lunalab_summit_xl_gen_description/meshes/kinova/v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
- link robot_j2s7s300_link_7: geometry collision mesh filename=package://lunalab_summit_xl_gen_description/meshes/kinova/c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; visual mesh filename=package://lunalab_summit_xl_gen_description/meshes/kinova/v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

File: lunalab_summit_xl_gen_description/urdf/manipulators/kinova/j2s7s300.xacro (robot description, xacro)
@@ -145,17 +145,17 @@
     <xacro:kinova_armlink link_name="${prefix}link_base" link_mesh="${link_base_mesh}" collision="${collision_arm}" mu="${link_base_mu}"/>
     <xacro:kinova_armjoint joint_name="${prefix}joint_base" type="${joint_base_type}" parent="${base_parent}" child="${prefix}link_base" joint_axis_xyz="${joint_base_axis_xyz}" joint_origin_xyz="${joint_base_origin_xyz}" joint_origin_rpy="${joint_base_origin_rpy}" joint_lower_limit="0" joint_upper_limit="0" joint_velocity_limit="0" joint_torque_limit="0" fixed="true" safety_limits="${safety_limits}" safety_position_margin="${safety_position_margin}" safety_k_position="${safety_k_position}" gazebo_preserve_fixed_joint="${gazebo_preserve_fixed_joint}"/>
-    <xacro:kinova_armlink link_name="${prefix}link_1" link_mesh="${link_1_mesh}" use_ring_mesh="true" collision="${collision_arm}" mu="${link_1_mu}"/>
+    <xacro:kinova_armlink link_name="${prefix}link_1" link_mesh="${link_1_mesh}" collision="${collision_arm}" mu="${link_1_mu}"/>
     <xacro:kinova_armjoint joint_name="${prefix}joint_1" type="${joint_1_type}" parent="${prefix}link_base" child="${prefix}link_1" joint_axis_xyz="${joint_1_axis_xyz}" joint_origin_xyz="${joint_1_origin_xyz}" joint_origin_rpy="${joint_1_origin_rpy}" joint_damping="${joint_1_damping}" joint_friction="${joint_1_friction}" joint_lower_limit="${joint_1_lower_limit}" joint_upper_limit="${joint_1_upper_limit}" joint_velocity_limit="${joint_1_velocity_limit}" joint_torque_limit="${joint_1_torque_limit}" safety_limits="${safety_limits}" safety_position_margin="${safety_position_margin}" safety_k_position="${safety_k_position}" gazebo_preserve_fixed_joint="${gazebo_preserve_fixed_joint}"/>
-    <xacro:kinova_armlink link_name="${prefix}link_2" link_mesh="${link_2_mesh}" use_ring_mesh="true" collision="${collision_arm}" mu="${link_2_mu}"/>
+    <xacro:kinova_armlink link_name="${prefix}link_2" link_mesh="${link_2_mesh}" collision="${collision_arm}" mu="${link_2_mu}"/>
     <xacro:kinova_armjoint joint_name="${prefix}joint_2" type="${joint_2_type}" parent="${prefix}link_1" child="${prefix}link_2" joint_axis_xyz="${joint_2_axis_xyz}" joint_origin_xyz="${joint_2_origin_xyz}" joint_origin_rpy="${joint_2_origin_rpy}" joint_damping="${joint_2_damping}" joint_friction="${joint_2_friction}" joint_lower_limit="${joint_2_lower_limit}" joint_upper_limit="${joint_2_upper_limit}" joint_velocity_limit="${joint_2_velocity_limit}" joint_torque_limit="${joint_2_torque_limit}" safety_limits="${safety_limits}" safety_position_margin="${safety_position_margin}" safety_k_position="${safety_k_position}" gazebo_preserve_fixed_joint="${gazebo_preserve_fixed_joint}"/>
-    <xacro:kinova_armlink link_name="${prefix}link_3" link_mesh="${link_3_mesh}" use_ring_mesh="true" collision="${collision_arm}" mu="${link_3_mu}"/>
+    <xacro:kinova_armlink link_name="${prefix}link_3" link_mesh="${link_3_mesh}" collision="${collision_arm}" mu="${link_3_mu}"/>
     <xacro:kinova_armjoint joint_name="${prefix}joint_3" type="${joint_3_type}" parent="${prefix}link_2" child="${prefix}link_3" joint_axis_xyz="${joint_3_axis_xyz}" joint_origin_xyz="${joint_3_origin_xyz}" joint_origin_rpy="${joint_3_origin_rpy}" joint_damping="${joint_3_damping}" joint_friction="${joint_3_friction}" joint_lower_limit="${joint_3_lower_limit}" joint_upper_limit="${joint_3_upper_limit}" joint_velocity_limit="${joint_3_velocity_limit}" joint_torque_limit="${joint_3_torque_limit}" safety_limits="${safety_limits}" safety_position_margin="${safety_position_margin}" safety_k_position="${safety_k_position}" gazebo_preserve_fixed_joint="${gazebo_preserve_fixed_joint}"/>
-    <xacro:kinova_armlink link_name="${prefix}link_4" link_mesh="${link_4_mesh}" use_ring_mesh="true" collision="${collision_arm}" mu="${link_4_mu}"/>
+    <xacro:kinova_armlink link_name="${prefix}link_4" link_mesh="${link_4_mesh}" collision="${collision_arm}" mu="${link_4_mu}"/>
     <xacro:kinova_armjoint joint_name="${prefix}joint_4" type="${joint_4_type}" parent="${prefix}link_3" child="${prefix}link_4" joint_axis_xyz="${joint_4_axis_xyz}" joint_origin_xyz="${joint_4_origin_xyz}" joint_origin_rpy="${joint_4_origin_rpy}" joint_damping="${joint_4_damping}" joint_friction="${joint_4_friction}" joint_lower_limit="${joint_4_lower_limit}" joint_upper_limit="${joint_4_upper_limit}" joint_velocity_limit="${joint_4_velocity_limit}" joint_torque_limit="${joint_4_torque_limit}" safety_limits="${safety_limits}" safety_position_margin="${safety_position_margin}" safety_k_position="${safety_k_position}" gazebo_preserve_fixed_joint="${gazebo_preserve_fixed_joint}"/>
-    <xacro:kinova_armlink link_name="${prefix}link_5" link_mesh="${link_5_mesh}" use_ring_mesh="true" ring_mesh="ring_small" collision="${collision_arm}" mu="${link_5_mu}"/>
+    <xacro:kinova_armlink link_name="${prefix}link_5" link_mesh="${link_5_mesh}" collision="${collision_arm}" mu="${link_5_mu}"/>
     <xacro:kinova_armjoint joint_name="${prefix}joint_5" type="${joint_5_type}" parent="${prefix}link_4" child="${prefix}link_5" joint_axis_xyz="${joint_5_axis_xyz}" joint_origin_xyz="${joint_5_origin_xyz}" joint_origin_rpy="${joint_5_origin_rpy}" joint_damping="${joint_5_damping}" joint_friction="${joint_5_friction}" joint_lower_limit="${joint_5_lower_limit}" joint_upper_limit="${joint_5_upper_limit}" joint_velocity_limit="${joint_5_velocity_limit}" joint_torque_limit="${joint_5_torque_limit}" safety_limits="${safety_limits}" safety_position_margin="${safety_position_margin}" safety_k_position="${safety_k_position}" gazebo_preserve_fixed_joint="${gazebo_preserve_fixed_joint}"/>
-    <xacro:kinova_armlink link_name="${prefix}link_6" link_mesh="${link_6_mesh}" use_ring_mesh="true" ring_mesh="ring_small" collision="${collision_arm}" mu="${link_6_mu}"/>
+    <xacro:kinova_armlink link_name="${prefix}link_6" link_mesh="${link_6_mesh}" collision="${collision_arm}" mu="${link_6_mu}"/>
     <xacro:kinova_armjoint joint_name="${prefix}joint_6" type="${joint_6_type}" parent="${prefix}link_5" child="${prefix}link_6" joint_axis_xyz="${joint_6_axis_xyz}" joint_origin_xyz="${joint_6_origin_xyz}" joint_origin_rpy="${joint_6_origin_rpy}" joint_damping="${joint_6_damping}" joint_friction="${joint_6_friction}" joint_lower_limit="${joint_6_lower_limit}" joint_upper_limit="${joint_6_upper_limit}" joint_velocity_limit="${joint_6_velocity_limit}" joint_torque_limit="${joint_6_torque_limit}" safety_limits="${safety_limits}" safety_position_margin="${safety_position_margin}" safety_k_position="${safety_k_position}" gazebo_preserve_fixed_joint="${gazebo_preserve_fixed_joint}"/>
-    <xacro:kinova_armlink link_name="${prefix}link_7" link_mesh="${link_7_mesh}" use_ring_mesh="true" ring_mesh="ring_small" collision="${collision_gripper}" mu="${link_7_mu}"/>
+    <xacro:kinova_armlink link_name="${prefix}link_7" link_mesh="${link_7_mesh}" collision="${collision_gripper}" mu="${link_7_mu}"/>
     <xacro:kinova_armjoint joint_name="${prefix}joint_7" type="${joint_7_type}" parent="${prefix}link_6" child="${prefix}link_7" joint_axis_xyz="${joint_7_axis_xyz}" joint_origin_xyz="${joint_7_origin_xyz}" joint_origin_rpy="${joint_7_origin_rpy}" joint_damping="${joint_7_damping}" joint_friction="${joint_7_friction}" joint_lower_limit="${joint_7_lower_limit}" joint_upper_limit="${joint_7_upper_limit}" joint_velocity_limit="${joint_7_velocity_limit}" joint_torque_limit="${joint_7_torque_limit}" safety_limits="${safety_limits}" safety_position_margin="${safety_position_margin}" safety_k_position="${safety_k_position}" gazebo_preserve_fixed_joint="${gazebo_preserve_fixed_joint}"/>
     <xacro:kinova_virtual_fixed_link joint_name="${prefix}joint_end_effector" parent="${prefix}link_7" child="${prefix}end_effector" joint_origin_xyz="${joint_end_effector_origin_xyz}" joint_origin_rpy="${joint_end_effector_origin_rpy}" gazebo_preserve_fixed_joint="${gazebo_preserve_fixed_joint}"/>

File: lunalab_summit_xl_gen_description/urdf/manipulators/kinova/kinova_common.xacro (robot description, xacro)
@@ -10,6 +10,4 @@
   <!-- link_name     - Name of the link to create -->
   <!-- link_mesh     - Name of the mesh to load (filename must be identical for visual and collision geometry, while located in their specific directories) -->
-  <!-- use_ring_mesh - Flag to enable ring mesh (visual only) -->
-  <!-- ring_mesh     - Selector of ring mesh type, which must correspond to mesh name, e.g. `ring_small` -->
   <!-- collision     - Flag to enable collision geometry -->
   <!-- mu            - Friction of the surface applied to both directions -->
@@ -17,6 +15,4 @@
     link_name
     link_mesh
-    use_ring_mesh:=false
-    ring_mesh:=ring_big
     collision:=true
     mu:=1.0
@@ -28,12 +24,4 @@
         </geometry>
       </visual>
-      <!-- Add ring to the link, if enabled -->
-      <xacro:if value="${use_ring_mesh}">
-        <visual>
-          <geometry>
-            <mesh filename="package://lunalab_summit_xl_gen_description/meshes/kinova/visual/${ring_mesh}.dae"/>
-          </geometry>
-        </visual>
-      </xacro:if>
       <xacro:if value="${collision}">
         <collision>
@@ -48,4 +36,19 @@
       <mu1 value="${mu}"/>
       <mu2 value="${mu}"/>
+    </gazebo>
+    <gazebo reference="${link_name}">
+      <visual>
+        <material>
+            <diffuse>1 1 1 1</diffuse>
+            <specular>1 1 1 1</specular>
+            <pbr>
+              <metal>
+                  <albedo_map>package://lunalab_summit_xl_gen_description/materials/textures/kinova/kinova_gen2_albedo.png</albedo_map>
+                  <roughness_map>package://lunalab_summit_xl_gen_description/materials/textures/kinova/kinova_gen2_roughness.png</roughness_map>
+                  <metalness_map>package://lunalab_summit_xl_gen_description/materials/textures/kinova/kinova_gen2_metalness.png</metalness_map>
+              </metal>
+            </pbr>
+        </material>
+      </visual>
     </gazebo>
   </xacro:macro>
@@ -93,5 +96,5 @@
       </xacro:if>
     </xacro:if>
-    <xacro:unless value="${type =='fixed'}">
+    <xacro:unless value="${type == 'fixed'}">
       <xacro:if value="${joint_velocity_limit == dummy_default_value}">
         <xacro:ERROR_joint_velocity_limit_needs_to_be_set_for_a_non_fixed_joint/>

File: lunalab_summit_xl_gen_description/urdf/summit_xl/summit_xl_base.xacro (robot description, xacro)
@@ -72,4 +72,19 @@
       </gazebo>
     </xacro:if>
+    <gazebo reference="${prefix}base_link">
+      <visual>
+        <material>
+            <diffuse>1 1 1 1</diffuse>
+            <specular>1 1 1 1</specular>
+            <pbr>
+              <metal>
+                  <albedo_map>package://lunalab_summit_xl_gen_description/materials/textures/summit_xl/chassis_albedo.png</albedo_map>
+                  <roughness_map>package://lunalab_summit_xl_gen_description/materials/textures/summit_xl/chassis_roughness.png</roughness_map>
+                  <metalness_map>package://lunalab_summit_xl_gen_description/materials/textures/summit_xl/chassis_metalness.png</metalness_map>
+              </metal>
+            </pbr>
+        </material>
+      </visual>
+    </gazebo>
   </xacro:macro>
 </robot>
