Commit message: Disable `base_docking_contact_link` not present in LunaLab variant
Signed-off-by: Andrej Orsula <orsula.andrej@gmail.com>

File: lunalab_summit_xl_gen_description/urdf/lunalab_summit_xl_gen.urdf (robot description, URDF)
Before this commit: robot lunalab_summit_xl_gen, 22 links, 21 joints
Links:
- removed link robot_summit_xl_base_docking_contact_link
Joints:
- removed joint robot_summit_xl_base_docking_joint

File: lunalab_summit_xl_gen_description/urdf/summit_xl/summit_xl_base.xacro (robot description, xacro)
@@ -53,5 +53,5 @@
       </xacro:if>
     </link>
-    <link name="${prefix}base_docking_contact_link">
+    <!-- <link name="${prefix}base_docking_contact_link">
       <xacro:if value="${gazebo_preserve_fixed_joint}">
         <inertial>
@@ -65,5 +65,5 @@
       <parent link="${prefix}base_link"/>
       <child link="${prefix}base_docking_contact_link"/>
-    </joint>
+    </joint> -->
     <xacro:if value="${gazebo_preserve_fixed_joint}">
       <gazebo reference="${prefix}base_docking_joint">
@@ -75,13 +75,13 @@
       <visual>
         <material>
-            <diffuse>1 1 1 1</diffuse>
-            <specular>1 1 1 1</specular>
-            <pbr>
-              <metal>
-                  <albedo_map>package://lunalab_summit_xl_gen_description/materials/textures/summit_xl/chassis_albedo.png</albedo_map>
-                  <roughness_map>package://lunalab_summit_xl_gen_description/materials/textures/summit_xl/chassis_roughness.png</roughness_map>
-                  <metalness_map>package://lunalab_summit_xl_gen_description/materials/textures/summit_xl/chassis_metalness.png</metalness_map>
-              </metal>
-            </pbr>
+          <diffuse>1 1 1 1</diffuse>
+          <specular>1 1 1 1</specular>
+          <pbr>
+            <metal>
+              <albedo_map>package://lunalab_summit_xl_gen_description/materials/textures/summit_xl/chassis_albedo.png</albedo_map>
+              <roughness_map>package://lunalab_summit_xl_gen_description/materials/textures/summit_xl/chassis_roughness.png</roughness_map>
+              <metalness_map>package://lunalab_summit_xl_gen_description/materials/textures/summit_xl/chassis_metalness.png</metalness_map>
+            </metal>
+          </pbr>
         </material>
       </visual>

Commit message: Update inertial properties of Summit XL base
Signed-off-by: Andrej Orsula <orsula.andrej@gmail.com>

File: lunalab_summit_xl_gen_description/urdf/lunalab_summit_xl_gen.urdf (robot description, URDF)
Before this commit: robot lunalab_summit_xl_gen, 21 links, 20 joints
Links:
- link robot_summit_xl_base_link: mass 25.0 -> 50.0

File: lunalab_summit_xl_gen_description/urdf/summit_xl/summit_xl_base.xacro (robot description, xacro)
@@ -34,7 +34,7 @@
     <link name="${prefix}base_link">
       <inertial>
-        <mass value="25.0"/>
-        <origin xyz="0 0 0"/>
-        <inertia ixx="1.391" ixy="0.004" ixz="0.0" iyy="6.853" iyz="0.0" izz="6.125"/>
+        <mass value="50.0"/>
+        <origin xyz="-0.0246066 -1.3125e-05 0.157214"/>
+        <inertia ixx="0.8773624360089227" ixy="-0.0001914814670566834" ixz="0.09929940455155015" iyy="1.739156928222513" iyz="2.9628167736189533e-05" izz="1.9022131402815483"/>
       </inertial>
       <visual>

Commit message: Reduce j2s7s300 joint limits
Signed-off-by: Andrej Orsula <orsula.andrej@gmail.com>

File: lunalab_summit_xl_gen_description/urdf/lunalab_summit_xl_gen.urdf (robot description, URDF)
Before this commit: robot lunalab_summit_xl_gen, 21 links, 20 joints
Joints:
- joint robot_j2s7s300_joint_1: limit lower=-174.04423300887453 upper=174.04423300887453 effort=40 velocity=0.6283185307179586 -> lower=-6.283185307179586 upper=6.283185307179586 effort=40 velocity=0.6283185307179586
- joint robot_j2s7s300_joint_3: limit lower=-174.04423300887453 upper=174.04423300887453 effort=40 velocity=0.6283185307179586 -> lower=-6.283185307179586 upper=6.283185307179586 effort=40 velocity=0.6283185307179586
- joint robot_j2s7s300_joint_5: limit lower=-174.04423300887453 upper=174.04423300887453 effort=20 velocity=0.8377580409572781 -> lower=-6.283185307179586 upper=6.283185307179586 effort=20 velocity=0.8377580409572781
- joint robot_j2s7s300_joint_7: limit lower=-174.04423300887453 upper=174.04423300887453 effort=20 velocity=0.8377580409572781 -> lower=-6.283185307179586 upper=6.283185307179586 effort=20 velocity=0.8377580409572781

File: lunalab_summit_xl_gen_description/urdf/manipulators/kinova/j2s7s300.xacro (robot description, xacro)
@@ -38,6 +38,6 @@
   <xacro:property name="joint_1_origin_xyz" value="0 0 0.15675"/>
   <xacro:property name="joint_1_origin_rpy" value="0 ${pi} 0"/>
-  <xacro:property name="joint_1_lower_limit" value="${-55.4*pi}"/>
-  <xacro:property name="joint_1_upper_limit" value="${55.4*pi}"/>
+  <xacro:property name="joint_1_lower_limit" value="${-2*pi}"/>
+  <xacro:property name="joint_1_upper_limit" value="${2*pi}"/>
   <xacro:property name="joint_1_velocity_limit" value="${36*pi/180}"/>
   <xacro:property name="joint_1_torque_limit" value="40"/>
@@ -60,6 +60,6 @@
   <xacro:property name="joint_3_origin_xyz" value="0 -0.205 0"/>
   <xacro:property name="joint_3_origin_rpy" value="-${pi/2} 0 0"/>
-  <xacro:property name="joint_3_lower_limit" value="${-55.4*pi}"/>
-  <xacro:property name="joint_3_upper_limit" value="${55.4*pi}"/>
+  <xacro:property name="joint_3_lower_limit" value="${-2*pi}"/>
+  <xacro:property name="joint_3_upper_limit" value="${2*pi}"/>
   <xacro:property name="joint_3_velocity_limit" value="${36*pi/180}"/>
   <xacro:property name="joint_3_torque_limit" value="40"/>
@@ -82,6 +82,6 @@
   <xacro:property name="joint_5_origin_xyz" value="0 0.2073 -0.0114"/>
   <xacro:property name="joint_5_origin_rpy" value="${-pi/2} 0 ${pi}"/>
-  <xacro:property name="joint_5_lower_limit" value="${-55.4*pi}"/>
-  <xacro:property name="joint_5_upper_limit" value="${55.4*pi}"/>
+  <xacro:property name="joint_5_lower_limit" value="${-2*pi}"/>
+  <xacro:property name="joint_5_upper_limit" value="${2*pi}"/>
   <xacro:property name="joint_5_velocity_limit" value="${48*pi/180}"/>
   <xacro:property name="joint_5_torque_limit" value="20"/>
@@ -104,6 +104,6 @@
   <xacro:property name="joint_7_origin_xyz" value="0 0.10375 0"/>
   <xacro:property name="joint_7_origin_rpy" value="${-pi/2} 0 ${pi}"/>
-  <xacro:property name="joint_7_lower_limit" value="${-55.4*pi}"/>
-  <xacro:property name="joint_7_upper_limit" value="${55.4*pi}"/>
+  <xacro:property name="joint_7_lower_limit" value="${-2*pi}"/>
+  <xacro:property name="joint_7_upper_limit" value="${2*pi}"/>
   <xacro:property name="joint_7_velocity_limit" value="${48*pi/180}"/>
   <xacro:property name="joint_7_torque_limit" value="20"/>
