Commit message: Change gripper move_group to use passive finger tip joints
Signed-off-by: Andrej Orsula <orsula.andrej@gmail.com>

File: lunalab_summit_xl_gen_moveit_config/srdf/lunalab_summit_xl_gen_j2s7s300.xacro (robot description, xacro)
@@ -19,13 +19,10 @@
     </group>
     <group name="gripper">
-      <link name="${prefix}j2s7s300_link_finger_1"/>
-      <link name="${prefix}j2s7s300_link_finger_tip_1"/>
-      <link name="${prefix}j2s7s300_link_finger_2"/>
-      <link name="${prefix}j2s7s300_link_finger_tip_2"/>
-      <link name="${prefix}j2s7s300_link_finger_3"/>
-      <link name="${prefix}j2s7s300_link_finger_tip_3"/>
       <joint name="${prefix}j2s7s300_joint_finger_1"/>
       <joint name="${prefix}j2s7s300_joint_finger_2"/>
       <joint name="${prefix}j2s7s300_joint_finger_3"/>
+      <passive_joint name="${prefix}j2s7s300_joint_finger_tip_1"/>
+      <passive_joint name="${prefix}j2s7s300_joint_finger_tip_2"/>
+      <passive_joint name="${prefix}j2s7s300_joint_finger_tip_3"/>
     </group>
     <group_state name="vertical" group="arm">
@@ -51,7 +48,4 @@
       <joint name="${prefix}j2s7s300_joint_finger_2" value="0.2"/>
       <joint name="${prefix}j2s7s300_joint_finger_3" value="0.2"/>
-      <joint name="robot_j2s7s300_joint_finger_tip_1" value="0.0"/>
-      <joint name="robot_j2s7s300_joint_finger_tip_2" value="0.0"/>
-      <joint name="robot_j2s7s300_joint_finger_tip_3" value="0.0"/>
     </group_state>
     <group_state name="close" group="gripper">
@@ -59,7 +53,4 @@
       <joint name="${prefix}j2s7s300_joint_finger_2" value="1.2"/>
       <joint name="${prefix}j2s7s300_joint_finger_3" value="1.2"/>
-      <joint name="robot_j2s7s300_joint_finger_tip_1" value="0.0"/>
-      <joint name="robot_j2s7s300_joint_finger_tip_2" value="0.0"/>
-      <joint name="robot_j2s7s300_joint_finger_tip_3" value="0.0"/>
     </group_state>
     <end_effector name="gripper" parent_link="${prefix}j2s7s300_end_effector" group="gripper" parent_group="arm"/>

Commit message: Update j2s7s300 joint positions and limits
Signed-off-by: Andrej Orsula <orsula.andrej@gmail.com>

File: lunalab_summit_xl_gen_moveit_config/srdf/lunalab_summit_xl_gen_j2s7s300.xacro (robot description, xacro)
@@ -37,9 +37,9 @@
     <group_state name="home" group="arm">
       <joint name="${prefix}j2s7s300_joint_1" value="0"/>
-      <joint name="${prefix}j2s7s300_joint_2" value="${200*pi/180}"/>
+      <joint name="${prefix}j2s7s300_joint_2" value="${pi}"/>
       <joint name="${prefix}j2s7s300_joint_3" value="0"/>
-      <joint name="${prefix}j2s7s300_joint_4" value="${300*pi/180}"/>
+      <joint name="${prefix}j2s7s300_joint_4" value="${270*pi/180}"/>
       <joint name="${prefix}j2s7s300_joint_5" value="0"/>
-      <joint name="${prefix}j2s7s300_joint_6" value="${100*pi/180}"/>
+      <joint name="${prefix}j2s7s300_joint_6" value="${90*pi/180}"/>
       <joint name="${prefix}j2s7s300_joint_7" value="0"/>
     </group_state>
