Commit message: Add joint friction and damping to wheels
Signed-off-by: Andrej Orsula <orsula.andrej@gmail.com>

File: lunalab_summit_xl_gen_description/urdf/summit_xl/rubber_wheel.xacro (robot description, xacro)
@@ -4,8 +4,15 @@
   <!-- Properties -->
   <!--            -->
-  <!-- Wheels -->
+  <!-- Link -->
   <xacro:property name="rubber_wheel_radius" value="0.11"/>
   <xacro:property name="rubber_wheel_width" value="0.15"/>
   <xacro:property name="rubber_wheel_mass" value="6.5"/>
+  <xacro:property name="rubber_wheel_mu1" value="1.9"/>
+  <xacro:property name="rubber_wheel_mu2" value="1.7"/>
+  <!-- Joint -->
+  <xacro:property name="rubber_wheel_effort_limit" value="100"/>
+  <xacro:property name="rubber_wheel_velocity_limit" value="100"/>
+  <xacro:property name="rubber_wheel_damping" value="0.035"/>
+  <xacro:property name="rubber_wheel_friction" value="0.0005"/>
   <!--       -->
   <!-- Macro -->
@@ -42,6 +49,6 @@
       <xacro:insert_block name="origin"/>
       <axis xyz="0 1 0" rpy="0 0 0"/>
-      <limit effort="100" velocity="100"/>
-      <joint_properties damping="0.0" friction="0.0"/>
+      <limit effort="${rubber_wheel_effort_limit}" velocity="${rubber_wheel_velocity_limit}"/>
+      <dynamics damping="${rubber_wheel_damping}" friction="${rubber_wheel_friction}"/>
     </joint>
     <link name="${prefix}wheel">
@@ -80,6 +87,6 @@
     </transmission>
     <gazebo reference="${prefix}wheel">
-      <mu1 value="1.9"/>
-      <mu2 value="1.7"/>
+      <mu1 value="${rubber_wheel_mu1}"/>
+      <mu2 value="${rubber_wheel_mu2}"/>
       <fdir1 value="1 0 0"/>
     </gazebo>

Commit message: Add PBR material for rubber wheels
Signed-off-by: Andrej Orsula <orsula.andrej@gmail.com>

File: lunalab_summit_xl_gen_description/urdf/summit_xl/rubber_wheel.xacro (robot description, xacro)
@@ -94,4 +94,20 @@
       <fdir1 value="1 0 0"/>
     </gazebo>
+    <gazebo reference="${prefix}wheel">
+      <visual>
+        <material>
+            <diffuse>1 1 1 1</diffuse>
+            <specular>1 1 1 1</specular>
+            <pbr>
+                <metal>
+                    <albedo_map>package://lunalab_summit_xl_gen_description/materials/textures/summit_xl/rubber_wheel_albedo.png</albedo_map>
+                    <normal_map>package://lunalab_summit_xl_gen_description/materials/textures/summit_xl/rubber_wheel_normal.png</normal_map>
+                    <roughness_map>package://lunalab_summit_xl_gen_description/materials/textures/summit_xl/rubber_wheel_roughness.png</roughness_map>
+                    <metalness_map>package://lunalab_summit_xl_gen_description/materials/textures/summit_xl/rubber_wheel_metalness.png</metalness_map>
+                </metal>
+            </pbr>
+        </material>
+      </visual>
+    </gazebo>
   </xacro:macro>
 </robot>
